Commit message: Added Front and Rear Bumper

File: urdf/junior.urdf (robot description, URDF)
Before this commit: robot Junior, 8 links, 7 joints
Links:
- added link BackBumper; visual mesh filename=package://junior_description/meshes/robitBackBumper.stl
- added link FrontBumper; visual mesh filename=package://junior_description/meshes/robitFrontBumper.stl
Joints:
- added joint BackBumperLoc: type fixed, parent Chassis, child BackBumper, origin xyz=-0.321 0 -0.0795 rpy=0 0 0
- added joint FrontBumperLoc: type fixed, parent Chassis, child FrontBumper, origin xyz=0.321 0 0.025 rpy=0 0 0
