Commit message: Fixed URI Mesh Errors for Gazebo

File: urdf/experimental.urdf.xacro (robot description, xacro)
@@ -13,5 +13,5 @@
 <!-- Front Lidar Length: 0.155m -->
 <!-- Front Lidar Height: 0.185m -->
-<robot name="Junior">
+<robot name="junior">
     <material name="black">
         <color rgba="0 0 0 1"/>
@@ -30,5 +30,5 @@
         <visual>
             <geometry>
-                <mesh filename="$(find junior_description)/meshes/robitChassis.stl"/>
+                <mesh filename="/home/csrobot/junior_ws/src/junior_description/meshes/robitChassis.stl"/>
             </geometry>
             <material name="red"/>
@@ -43,5 +43,5 @@
         <visual>
             <geometry>
-                <mesh filename="$(find junior_description)/meshes/robitFrontBumper.stl"/>
+                <mesh filename="/home/csrobot/junior_ws/src/junior_description/meshes/robitFrontBumper.stl"/>
             </geometry>
             <material name="black"/>
@@ -56,5 +56,5 @@
         <visual>
             <geometry>
-                <mesh filename="$(find junior_description)/meshes/robitBackBumper.stl"/>
+                <mesh filename="/home/csrobot/junior_ws/src/junior_description/meshes/robitBackBumper.stl"/>
             </geometry>
             <material name="black"/>
@@ -69,5 +69,5 @@
         <visual>
             <geometry>
-                <mesh filename="$(find junior_description)/meshes/robitFrontLidarCase.stl"/>
+                <mesh filename="/home/csrobot/junior_ws/src/junior_description/meshes/robitFrontLidarCase.stl"/>
             </geometry>
             <material name="skyblue"/>
@@ -82,5 +82,5 @@
         <visual>
             <geometry>
-                <mesh filename="$(find junior_description)/meshes/robitFrontLidarGlass.stl"/>
+                <mesh filename="/home/csrobot/junior_ws/src/junior_description/meshes/robitFrontLidarGlass.stl"/>
             </geometry>
             <material name="black"/>
@@ -95,5 +95,5 @@
         <visual>
             <geometry>
-                <mesh filename="$(find junior_description)/meshes/robitWheel.stl"/>
+                <mesh filename="/home/csrobot/junior_ws/src/junior_description/meshes/robitWheel.stl"/>
             </geometry>
             <material name="black"/>
@@ -108,5 +108,5 @@
         <visual>
             <geometry>
-                <mesh filename="$(find junior_description)/meshes/robitWheel.stl"/>
+                <mesh filename="/home/csrobot/junior_ws/src/junior_description/meshes/robitWheel.stl"/>
             </geometry>
             <material name="black"/>
@@ -121,5 +121,5 @@
         <visual>
             <geometry>
-                <mesh filename="$(find junior_description)/meshes/robitWheel.stl"/>
+                <mesh filename="/home/csrobot/junior_ws/src/junior_description/meshes/robitWheel.stl"/>
             </geometry>
             <material name="black"/>
@@ -134,5 +134,5 @@
         <visual>
             <geometry>
-                <mesh filename="$(find junior_description)/meshes/robitWheel.stl"/>
+                <mesh filename="/home/csrobot/junior_ws/src/junior_description/meshes/robitWheel.stl"/>
             </geometry>
             <material name="black"/>
@@ -195,5 +195,5 @@
     <!-- END OF JOINTS -->
     <!-- Back bumper offset, required z amount to be at bottom of chassis and length / 2 for x-->
-    <!-- Experimentation with Moving Parts ex. Lidars, Wheels
+    <!--
     <gazebo reference="FrontLidarGlass">
         <sensor name="laser" type="ray">

Commit message: Working Gazebo Simulation with Paperweight Junior

File: urdf/experimental.urdf.xacro (robot description, xacro)
@@ -34,6 +34,12 @@
             <material name="red"/>
         </visual>
-        <inertial>
-            <mass value="10"/>
+        <collision>
+            <geometry>
+                <mesh filename="/home/csrobot/junior_ws/src/junior_description/meshes/robitChassis.stl"/>
+            </geometry>
+            <material name="red"/>
+        </collision>
+        <inertial>
+            <mass value="0.01"/>
             <inertia ixx="0.4" ixy="0.0" ixz="0.0" iyy="0.4" iyz="0.0" izz="0.2"/>
         </inertial>
@@ -47,6 +53,12 @@
             <material name="black"/>
         </visual>
-        <inertial>
-            <mass value="10"/>
+        <collision>
+            <geometry>
+                <mesh filename="/home/csrobot/junior_ws/src/junior_description/meshes/robitFrontBumper.stl"/>
+            </geometry>
+            <material name="black"/>
+        </collision>
+        <inertial>
+            <mass value="0.01"/>
             <inertia ixx="0.4" ixy="0.0" ixz="0.0" iyy="0.4" iyz="0.0" izz="0.2"/>
         </inertial>
@@ -60,6 +72,12 @@
             <material name="black"/>
         </visual>
-        <inertial>
-            <mass value="10"/>
+        <collision>
+            <geometry>
+                <mesh filename="/home/csrobot/junior_ws/src/junior_description/meshes/robitBackBumper.stl"/>
+            </geometry>
+            <material name="black"/>
+        </collision>
+        <inertial>
+            <mass value="0.01"/>
             <inertia ixx="0.4" ixy="0.0" ixz="0.0" iyy="0.4" iyz="0.0" izz="0.2"/>
         </inertial>
@@ -73,6 +91,12 @@
             <material name="skyblue"/>
         </visual>
-        <inertial>
-            <mass value="10"/>
+        <collision>
+            <geometry>
+                <mesh filename="/home/csrobot/junior_ws/src/junior_description/meshes/robitFrontLidarCase.stl"/>
+            </geometry>
+            <material name="skyblue"/>
+        </collision>
+        <inertial>
+            <mass value="0.01"/>
             <inertia ixx="0.4" ixy="0.0" ixz="0.0" iyy="0.4" iyz="0.0" izz="0.2"/>
         </inertial>
@@ -86,6 +110,12 @@
             <material name="black"/>
         </visual>
-        <inertial>
-            <mass value="10"/>
+        <collision>
+            <geometry>
+                <mesh filename="/home/csrobot/junior_ws/src/junior_description/meshes/robitFrontLidarGlass.stl"/>
+            </geometry>
+            <material name="black"/>
+        </collision>
+        <inertial>
+            <mass value="0.01"/>
             <inertia ixx="0.4" ixy="0.0" ixz="0.0" iyy="0.4" iyz="0.0" izz="0.2"/>
         </inertial>
@@ -99,6 +129,12 @@
             <material name="black"/>
         </visual>
-        <inertial>
-            <mass value="10"/>
+        <collision>
+            <geometry>
+                <mesh filename="/home/csrobot/junior_ws/src/junior_description/meshes/robitWheel.stl"/>
+            </geometry>
+            <material name="black"/>
+        </collision>
+        <inertial>
+            <mass value="0.01"/>
             <inertia ixx="0.4" ixy="0.0" ixz="0.0" iyy="0.4" iyz="0.0" izz="0.2"/>
         </inertial>
@@ -112,6 +148,12 @@
             <material name="black"/>
         </visual>
-        <inertial>
-            <mass value="10"/>
+        <collision>
+            <geometry>
+                <mesh filename="/home/csrobot/junior_ws/src/junior_description/meshes/robitWheel.stl"/>
+            </geometry>
+            <material name="black"/>
+        </collision>
+        <inertial>
+            <mass value="0.01"/>
             <inertia ixx="0.4" ixy="0.0" ixz="0.0" iyy="0.4" iyz="0.0" izz="0.2"/>
         </inertial>
@@ -125,6 +167,12 @@
             <material name="black"/>
         </visual>
-        <inertial>
-            <mass value="10"/>
+        <collision>
+            <geometry>
+                <mesh filename="/home/csrobot/junior_ws/src/junior_description/meshes/robitWheel.stl"/>
+            </geometry>
+            <material name="black"/>
+        </collision>
+        <inertial>
+            <mass value="0.01"/>
             <inertia ixx="0.4" ixy="0.0" ixz="0.0" iyy="0.4" iyz="0.0" izz="0.2"/>
         </inertial>
@@ -138,6 +186,12 @@
             <material name="black"/>
         </visual>
-        <inertial>
-            <mass value="10"/>
+        <collision>
+            <geometry>
+                <mesh filename="/home/csrobot/junior_ws/src/junior_description/meshes/robitWheel.stl"/>
+            </geometry>
+            <material name="black"/>
+        </collision>
+        <inertial>
+            <mass value="0.01"/>
             <inertia ixx="0.4" ixy="0.0" ixz="0.0" iyy="0.4" iyz="0.0" izz="0.2"/>
         </inertial>
@@ -147,5 +201,5 @@
         <parent link="base_link"/>
         <child link="Chassis"/>
-        <origin xyz="1 0 0.23"/>
+        <origin xyz="0 0 0.23"/>
     </joint>
     <joint name="FrontLidarHolster" type="fixed">

Commit message: Added Approx Mass and Created Working LaserScan for Front Lidar

File: urdf/experimental.urdf.xacro (robot description, xacro)
@@ -41,5 +41,5 @@
         </collision>
         <inertial>
-            <mass value="0.01"/>
+            <mass value="35"/>
             <inertia ixx="0.4" ixy="0.0" ixz="0.0" iyy="0.4" iyz="0.0" izz="0.2"/>
         </inertial>
@@ -60,5 +60,5 @@
         </collision>
         <inertial>
-            <mass value="0.01"/>
+            <mass value="3"/>
             <inertia ixx="0.4" ixy="0.0" ixz="0.0" iyy="0.4" iyz="0.0" izz="0.2"/>
         </inertial>
@@ -79,5 +79,5 @@
         </collision>
         <inertial>
-            <mass value="0.01"/>
+            <mass value="1.5"/>
             <inertia ixx="0.4" ixy="0.0" ixz="0.0" iyy="0.4" iyz="0.0" izz="0.2"/>
         </inertial>
@@ -98,5 +98,5 @@
         </collision>
         <inertial>
-            <mass value="0.01"/>
+            <mass value="2"/>
             <inertia ixx="0.4" ixy="0.0" ixz="0.0" iyy="0.4" iyz="0.0" izz="0.2"/>
         </inertial>
@@ -117,5 +117,5 @@
         </collision>
         <inertial>
-            <mass value="0.01"/>
+            <mass value="0.1"/>
             <inertia ixx="0.4" ixy="0.0" ixz="0.0" iyy="0.4" iyz="0.0" izz="0.2"/>
         </inertial>
@@ -136,5 +136,5 @@
         </collision>
         <inertial>
-            <mass value="0.01"/>
+            <mass value="5"/>
             <inertia ixx="0.4" ixy="0.0" ixz="0.0" iyy="0.4" iyz="0.0" izz="0.2"/>
         </inertial>
@@ -155,5 +155,5 @@
         </collision>
         <inertial>
-            <mass value="0.01"/>
+            <mass value="5"/>
             <inertia ixx="0.4" ixy="0.0" ixz="0.0" iyy="0.4" iyz="0.0" izz="0.2"/>
         </inertial>
@@ -174,5 +174,5 @@
         </collision>
         <inertial>
-            <mass value="0.01"/>
+            <mass value="5"/>
             <inertia ixx="0.4" ixy="0.0" ixz="0.0" iyy="0.4" iyz="0.0" izz="0.2"/>
         </inertial>
@@ -193,5 +193,5 @@
         </collision>
         <inertial>
-            <mass value="0.01"/>
+            <mass value="5"/>
             <inertia ixx="0.4" ixy="0.0" ixz="0.0" iyy="0.4" iyz="0.0" izz="0.2"/>
         </inertial>
@@ -249,5 +249,4 @@
     <!-- END OF JOINTS -->
     <!-- Back bumper offset, required z amount to be at bottom of chassis and length / 2 for x-->
-    <!--
     <gazebo reference="FrontLidarGlass">
         <sensor name="laser" type="ray">
@@ -277,4 +276,4 @@
             </plugin>
         </sensor>
-    </gazebo> -->
+    </gazebo>
 </robot>
