Commit message: Working Junior in RVIZ and Gazebo

File: urdf/junior.urdf.xacro (robot description, xacro)
@@ -1,16 +1,3 @@
 <?xml version="1.0"?>
-<!-- Chassis Width: 0.387m -->
-<!-- Chassis Length: 0.642m -->
-<!-- Chassis Height: 0.224m -->
-<!-- Wheel Diameter: 0.315m -->
-<!-- Wheel Width: 0.105m -->
-<!-- Wheel to Body: 0.125m -->
-<!-- Axle Distance: 0.386m -->
-<!-- Calculation 1: 0.1185m (0.237 / 2) -->
-<!-- Calculation 2: 0.193m (0.386 / 2) -->
-<!-- Calculation 3: 0.2635m (0.387 / 2 + 0.07) -->
-<!-- Front Lidar Width: 0.155m -->
-<!-- Front Lidar Length: 0.155m -->
-<!-- Front Lidar Height: 0.185m -->
 <robot name="junior">
     <material name="black">
@@ -30,5 +17,5 @@
         <visual>
             <geometry>
-                <mesh filename="/home/csrobot/junior_ws/src/junior_description/meshes/robitChassis.stl"/>
+                <mesh filename="file://$(find junior_description)/meshes/robitChassis.stl"/>
             </geometry>
             <material name="red"/>
@@ -36,5 +23,5 @@
         <collision>
             <geometry>
-                <mesh filename="/home/csrobot/junior_ws/src/junior_description/meshes/robitChassis.stl"/>
+                <mesh filename="file://$(find junior_description)/meshes/robitChassis.stl"/>
             </geometry>
             <material name="red"/>
@@ -49,11 +36,11 @@
         <visual>
             <geometry>
-                <mesh filename="/home/csrobot/junior_ws/src/junior_description/meshes/robitFrontBumper.stl"/>
-            </geometry>
-            <material name="black"/>
-        </visual>
-        <collision>
-            <geometry>
-                <mesh filename="/home/csrobot/junior_ws/src/junior_description/meshes/robitFrontBumper.stl"/>
+                <mesh filename="file://$(find junior_description)/meshes/robitFrontBumper.stl"/>
+            </geometry>
+            <material name="black"/>
+        </visual>
+        <collision>
+            <geometry>
+                <mesh filename="file://$(find junior_description)/meshes/robitFrontBumper.stl"/>
             </geometry>
             <material name="black"/>
@@ -68,11 +55,11 @@
         <visual>
             <geometry>
-                <mesh filename="/home/csrobot/junior_ws/src/junior_description/meshes/robitBackBumper.stl"/>
-            </geometry>
-            <material name="black"/>
-        </visual>
-        <collision>
-            <geometry>
-                <mesh filename="/home/csrobot/junior_ws/src/junior_description/meshes/robitBackBumper.stl"/>
+                <mesh filename="file://$(find junior_description)/meshes/robitBackBumper.stl"/>
+            </geometry>
+            <material name="black"/>
+        </visual>
+        <collision>
+            <geometry>
+                <mesh filename="file://$(find junior_description)/meshes/robitBackBumper.stl"/>
             </geometry>
             <material name="black"/>
@@ -87,5 +74,5 @@
         <visual>
             <geometry>
-                <mesh filename="/home/csrobot/junior_ws/src/junior_description/meshes/robitFrontLidarCase.stl"/>
+                <mesh filename="file://$(find junior_description)/meshes/robitFrontLidarCase.stl"/>
             </geometry>
             <material name="skyblue"/>
@@ -93,5 +80,5 @@
         <collision>
             <geometry>
-                <mesh filename="/home/csrobot/junior_ws/src/junior_description/meshes/robitFrontLidarCase.stl"/>
+                <mesh filename="file://$(find junior_description)/meshes/robitFrontLidarCase.stl"/>
             </geometry>
             <material name="skyblue"/>
@@ -106,11 +93,11 @@
         <visual>
             <geometry>
-                <mesh filename="/home/csrobot/junior_ws/src/junior_description/meshes/robitFrontLidarGlass.stl"/>
-            </geometry>
-            <material name="black"/>
-        </visual>
-        <collision>
-            <geometry>
-                <mesh filename="/home/csrobot/junior_ws/src/junior_description/meshes/robitFrontLidarGlass.stl"/>
+                <mesh filename="file://$(find junior_description)/meshes/robitFrontLidarGlass.stl"/>
+            </geometry>
+            <material name="black"/>
+        </visual>
+        <collision>
+            <geometry>
+                <mesh filename="file://$(find junior_description)/meshes/robitFrontLidarGlass.stl"/>
             </geometry>
             <material name="black"/>
@@ -125,11 +112,11 @@
         <visual>
             <geometry>
-                <mesh filename="/home/csrobot/junior_ws/src/junior_description/meshes/robitWheel.stl"/>
-            </geometry>
-            <material name="black"/>
-        </visual>
-        <collision>
-            <geometry>
-                <mesh filename="/home/csrobot/junior_ws/src/junior_description/meshes/robitWheel.stl"/>
+                <mesh filename="file://$(find junior_description)/meshes/robitWheel.stl"/>
+            </geometry>
+            <material name="black"/>
+        </visual>
+        <collision>
+            <geometry>
+                <mesh filename="file://$(find junior_description)/meshes/robitWheel.stl"/>
             </geometry>
             <material name="black"/>
@@ -144,11 +131,11 @@
         <visual>
             <geometry>
-                <mesh filename="/home/csrobot/junior_ws/src/junior_description/meshes/robitWheel.stl"/>
-            </geometry>
-            <material name="black"/>
-        </visual>
-        <collision>
-            <geometry>
-                <mesh filename="/home/csrobot/junior_ws/src/junior_description/meshes/robitWheel.stl"/>
+                <mesh filename="file://$(find junior_description)/meshes/robitWheel.stl"/>
+            </geometry>
+            <material name="black"/>
+        </visual>
+        <collision>
+            <geometry>
+                <mesh filename="file://$(find junior_description)/meshes/robitWheel.stl"/>
             </geometry>
             <material name="black"/>
@@ -163,11 +150,11 @@
         <visual>
             <geometry>
-                <mesh filename="/home/csrobot/junior_ws/src/junior_description/meshes/robitWheel.stl"/>
-            </geometry>
-            <material name="black"/>
-        </visual>
-        <collision>
-            <geometry>
-                <mesh filename="/home/csrobot/junior_ws/src/junior_description/meshes/robitWheel.stl"/>
+                <mesh filename="file://$(find junior_description)/meshes/robitWheel.stl"/>
+            </geometry>
+            <material name="black"/>
+        </visual>
+        <collision>
+            <geometry>
+                <mesh filename="file://$(find junior_description)/meshes/robitWheel.stl"/>
             </geometry>
             <material name="black"/>
@@ -182,11 +169,11 @@
         <visual>
             <geometry>
-                <mesh filename="/home/csrobot/junior_ws/src/junior_description/meshes/robitWheel.stl"/>
-            </geometry>
-            <material name="black"/>
-        </visual>
-        <collision>
-            <geometry>
-                <mesh filename="/home/csrobot/junior_ws/src/junior_description/meshes/robitWheel.stl"/>
+                <mesh filename="file://$(find junior_description)/meshes/robitWheel.stl"/>
+            </geometry>
+            <material name="black"/>
+        </visual>
+        <collision>
+            <geometry>
+                <mesh filename="file://$(find junior_description)/meshes/robitWheel.stl"/>
             </geometry>
             <material name="black"/>
@@ -248,5 +235,22 @@
     </joint>
     <!-- END OF JOINTS -->
-    <!-- Back bumper offset, required z amount to be at bottom of chassis and length / 2 for x-->
+    <!-- START OF GAZEBO -->
+    <!-- Chassis -->
+    <gazebo reference="Chassis">
+        <material>Gazebo/Red</material>
+    </gazebo>
+    <!-- Front Bumper -->
+    <gazebo reference="FrontBumper">
+        <material>Gazebo/Black</material>
+    </gazebo>
+    <!-- Back Bumper -->
+    <gazebo reference="BackBumper">
+        <material>Gazebo/Black</material>
+    </gazebo>
+    <!-- Front Lidar Case -->
+    <gazebo reference="FrontLidar">
+        <material>Gazebo/SkyBlue</material>
+    </gazebo>
+    <!-- Front Lidar -->
     <gazebo reference="FrontLidarGlass">
         <sensor name="laser" type="ray">
@@ -263,7 +267,6 @@
                 </scan>
                 <range>
-                    Range Unknown as of Now, Using Default Values
                     <min>0.3</min>
-                    <max>12</max>
+                    <max>5</max>
                 </range>
             </ray>
@@ -276,4 +279,20 @@
             </plugin>
         </sensor>
-    </gazebo>
+        <material>Gazebo/Black</material>
+    </gazebo>
+    <!-- WHEELS -->
+    <gazebo reference="WheelLeftFront">
+        <material>Gazebo/Black</material>
+    </gazebo>
+    <gazebo reference="WheelRightFront">
+        <material>Gazebo/Black</material>
+    </gazebo>
+    <gazebo reference="WheelLeftBack">
+        <material>Gazebo/Black</material>
+    </gazebo>
+    <gazebo reference="WheelRightBack">
+        <material>Gazebo/Black</material>
+    </gazebo>
+    <!-- END OF WHEELS -->
+    <!-- END OF GAZEBO -->
 </robot>

Commit message: Started Back Lidar Construction

File: urdf/junior.urdf.xacro (robot description, xacro)
@@ -108,4 +108,23 @@
         </inertial>
     </link>
+    <!-- Back Lidar Case Link -->
+    <link name="BackLidarCase">
+        <visual>
+            <geometry>
+                <mesh filename="file://$(find junior_description)/meshes/robitBackLidarCase.stl"/>
+            </geometry>
+            <material name="black"/>
+        </visual>
+        <collision>
+            <geometry>
+                <mesh filename="file://$(find junior_description)/meshes/robitBackLidarCase.stl"/>
+            </geometry>
+            <material name="black"/>
+        </collision>
+        <inertial>
+            <mass value="2"/>
+            <inertia ixx="0.4" ixy="0.0" ixz="0.0" iyy="0.4" iyz="0.0" izz="0.2"/>
+        </inertial>
+    </link>
     <!-- Left Front Link -->
     <link name="WheelLeftFront">
@@ -199,4 +218,9 @@
         <child link="FrontLidarGlass"/>
         <origin xyz="0.075 0 0"/>
+    </joint>
+    <joint name="BackLidarHolster" type="fixed">
+        <parent link="Chassis"/>
+        <child link="BackLidarCase"/>
+        <origin xyz="-0.285 0 0.319"/>
     </joint>
     <joint name="AxleLeftFront" type="continuous">

Commit message: Added Better Color/Material Quality

File: urdf/junior.urdf.xacro (robot description, xacro)
@@ -262,17 +262,41 @@
     <!-- Chassis -->
     <gazebo reference="Chassis">
-        <material>Gazebo/Red</material>
+        <visual>
+            <material>
+                <diffuse>1 0 0 1</diffuse>
+                <ambient>0.4 0.05 0.05 1</ambient>
+                <emissive>0 0 0 0</emissive>
+            </material>
+        </visual>
     </gazebo>
     <!-- Front Bumper -->
     <gazebo reference="FrontBumper">
-        <material>Gazebo/Black</material>
+        <visual>
+            <material>
+                <diffuse>0.2 0.2 0.2 1</diffuse>
+                <ambient>0.1 0.1 0.1 1</ambient>
+                <emissive>0 0 0 0</emissive>
+            </material>
+        </visual>
     </gazebo>
     <!-- Back Bumper -->
     <gazebo reference="BackBumper">
-        <material>Gazebo/Black</material>
+        <visual>
+            <material>
+                <diffuse>0.2 0.2 0.2 1</diffuse>
+                <ambient>0.1 0.1 0.1 1</ambient>
+                <emissive>0 0 0 0</emissive>
+            </material>
+        </visual>
     </gazebo>
     <!-- Front Lidar Case -->
     <gazebo reference="FrontLidar">
-        <material>Gazebo/SkyBlue</material>
+        <visual>
+            <material>
+                <diffuse>0.1 0.5 1 1</diffuse>
+                <ambient>0.0666 0.333 0.4 1</ambient>
+                <emissive>0 0 0 0</emissive>
+            </material>
+        </visual>
     </gazebo>
     <!-- Front Lidar -->
@@ -303,18 +327,48 @@
             </plugin>
         </sensor>
-        <material>Gazebo/Black</material>
+        <visual>
+            <material>
+                <diffuse>0.2 0.2 0.2 1</diffuse>
+                <ambient>0.1 0.1 0.1 1</ambient>
+                <emissive>0 0 0 0</emissive>
+            </material>
+        </visual>
     </gazebo>
     <!-- WHEELS -->
     <gazebo reference="WheelLeftFront">
-        <material>Gazebo/Black</material>
+        <visual>
+            <material>
+                <diffuse>0.2 0.2 0.2 1</diffuse>
+                <ambient>0.1 0.1 0.1 1</ambient>
+                <emissive>0 0 0 0</emissive>
+            </material>
+        </visual>
     </gazebo>
     <gazebo reference="WheelRightFront">
-        <material>Gazebo/Black</material>
+        <visual>
+            <material>
+                <diffuse>0.2 0.2 0.2 1</diffuse>
+                <ambient>0.1 0.1 0.1 1</ambient>
+                <emissive>0 0 0 0</emissive>
+            </material>
+        </visual>
     </gazebo>
     <gazebo reference="WheelLeftBack">
-        <material>Gazebo/Black</material>
+        <visual>
+            <material>
+                <diffuse>0.2 0.2 0.2 1</diffuse>
+                <ambient>0.1 0.1 0.1 1</ambient>
+                <emissive>0 0 0 0</emissive>
+            </material>
+        </visual>
     </gazebo>
     <gazebo reference="WheelRightBack">
-        <material>Gazebo/Black</material>
+        <visual>
+            <material>
+                <diffuse>0.2 0.2 0.2 1</diffuse>
+                <ambient>0.1 0.1 0.1 1</ambient>
+                <emissive>0 0 0 0</emissive>
+            </material>
+        </visual>
     </gazebo>
     <!-- END OF WHEELS -->

Commit message: Both Lidars Functioning in Gazebo

File: urdf/junior.urdf.xacro (robot description, xacro)
@@ -8,5 +8,8 @@
     </material>
     <material name="skyblue">
-        <color rgba="0.0 0.75 1.0 1.0"/>
+        <color rgba="0 0.75 1 1"/>
+    </material>
+    <material name="silver">
+        <color rgba="0.77 0.78 0.78 1"/>
     </material>
     <!-- Base Link -->
@@ -124,4 +127,42 @@
         <inertial>
             <mass value="2"/>
+            <inertia ixx="0.4" ixy="0.0" ixz="0.0" iyy="0.4" iyz="0.0" izz="0.2"/>
+        </inertial>
+    </link>
+    <!-- Back Lidar Stand Link -->
+    <link name="BackLidarStand">
+        <visual>
+            <geometry>
+                <mesh filename="file://$(find junior_description)/meshes/robitBackLidarStand.stl"/>
+            </geometry>
+            <material name="silver"/>
+        </visual>
+        <collision>
+            <geometry>
+                <mesh filename="file://$(find junior_description)/meshes/robitBackLidarStand.stl"/>
+            </geometry>
+            <material name="silver"/>
+        </collision>
+        <inertial>
+            <mass value="1"/>
+            <inertia ixx="0.4" ixy="0.0" ixz="0.0" iyy="0.4" iyz="0.0" izz="0.2"/>
+        </inertial>
+    </link>
+    <!-- Back Lidar Head -->
+    <link name="BackLidarHead">
+        <visual>
+            <geometry>
+                <mesh filename="file://$(find junior_description)/meshes/robitBackLidarHead.stl"/>
+            </geometry>
+            <material name="silver"/>
+        </visual>
+        <collision>
+            <geometry>
+                <mesh filename="file://$(find junior_description)/meshes/robitBackLidarHead.stl"/>
+            </geometry>
+            <material name="silver"/>
+        </collision>
+        <inertial>
+            <mass value="3"/>
             <inertia ixx="0.4" ixy="0.0" ixz="0.0" iyy="0.4" iyz="0.0" izz="0.2"/>
         </inertial>
@@ -223,4 +264,16 @@
         <child link="BackLidarCase"/>
         <origin xyz="-0.285 0 0.319"/>
+    </joint>
+    <joint name="BackLidarStandJoint" type="revolute">
+        <parent link="BackLidarCase"/>
+        <child link="BackLidarStand"/>
+        <origin xyz="0 0 -0.03"/>
+        <axis xyz="0 0 1"/>
+        <limit lower="-1" upper="1" effort="5" velocity="2"/>
+    </joint>
+    <joint name="BackLidarHeadJoint" type="fixed">
+        <parent link="BackLidarStand"/>
+        <child link="BackLidarHead"/>
+        <origin xyz="0 0 0.05" rpy="0 -3.14 0"/>
     </joint>
     <joint name="AxleLeftFront" type="continuous">
@@ -309,12 +362,12 @@
                 <scan>
                     <horizontal>
-                    <samples>270</samples>
-                    <min_angle>-2.35</min_angle>
-                    <max_angle>2.35</max_angle>
+                    <samples>360</samples>
+                    <min_angle>-1.57</min_angle>
+                    <max_angle>1.57</max_angle>
                     </horizontal>
                 </scan>
                 <range>
-                    <min>0.3</min>
-                    <max>5</max>
+                    <min>0.2</min>
+                    <max>3</max>
                 </range>
             </ray>
@@ -335,4 +388,59 @@
         </visual>
     </gazebo>
+    <!-- Back Lidar Case -->
+    <gazebo reference="BackLidarCase">
+        <visual>
+            <material>
+                <diffuse>0.2 0.2 0.2 1</diffuse>
+                <ambient>0.1 0.1 0.1 1</ambient>
+                <emissive>0 0 0 0</emissive>
+            </material>
+        </visual>
+    </gazebo>
+    <!-- Back Lidar Stand -->
+    <gazebo reference="BackLidarStand">
+        <visual>
+            <material>
+                <diffuse>0.77 0.78 0.78 1</diffuse>
+                <ambient>0.385 0.39 0.39 1</ambient>
+                <emissive>0 0 0 0</emissive>
+            </material>
+        </visual>
+    </gazebo>
+    <!-- Back Lidar Head -->
+    <gazebo reference="BackLidarHead">
+        <sensor name="blaser" type="ray">
+            <pose> 0 0 0 0 0 </pose>
+            <visualize>true</visualize>
+            <update_rate>10</update_rate>
+            <ray>
+                <scan>
+                    <horizontal>
+                    <samples>120</samples>
+                    <min_angle>-0.52</min_angle>
+                    <max_angle>0.52</max_angle>
+                    </horizontal>
+                </scan>
+                <range>
+                    <min>0.1</min>
+                    <max>2</max>
+                </range>
+            </ray>
+            <plugin name="bl_controller" filename="libgazebo_ros_ray_sensor.so">
+                <ros>
+                    <argument>-/out:=scan</argument>
+                </ros>
+                <output_type>sensor_msgs/LaserScan</output_type>
+                <frame_name>BackLidarHead</frame_name>
+            </plugin>
+        </sensor>
+        <visual>
+            <material>
+                <diffuse>0.77 0.78 0.78 1</diffuse>
+                <ambient>0.385 0.39 0.39 1</ambient>
+                <emissive>0 0 0 0</emissive>
+            </material>
+        </visual>
+    </gazebo>
     <!-- WHEELS -->
     <gazebo reference="WheelLeftFront">

Commit message: Updated Visual Chassis and Back Lidar Case

File: urdf/junior.urdf.xacro (robot description, xacro)
@@ -20,5 +20,5 @@
         <visual>
             <geometry>
-                <mesh filename="file://$(find junior_description)/meshes/robitChassis.stl"/>
+                <mesh filename="file://$(find junior_description)/meshes/robitChassisVisual.stl"/>
             </geometry>
             <material name="red"/>
@@ -164,5 +164,5 @@
         </collision>
         <inertial>
-            <mass value="3"/>
+            <mass value="5"/>
             <inertia ixx="0.4" ixy="0.0" ixz="0.0" iyy="0.4" iyz="0.0" izz="0.2"/>
         </inertial>
@@ -268,12 +268,15 @@
         <parent link="BackLidarCase"/>
         <child link="BackLidarStand"/>
-        <origin xyz="0 0 -0.03"/>
+        <origin xyz="0 0 -0.045"/>
         <axis xyz="0 0 1"/>
         <limit lower="-1" upper="1" effort="5" velocity="2"/>
     </joint>
-    <joint name="BackLidarHeadJoint" type="fixed">
+    <joint name="BackLidarHeadJoint" type="revolute">
         <parent link="BackLidarStand"/>
         <child link="BackLidarHead"/>
         <origin xyz="0 0 0.05" rpy="0 -3.14 0"/>
+        <axis xyz="0 1 0"/>
+        <dynamics damping="0" friction="0.75"/>
+        <limit lower="-1" upper="1" effort="5" velocity="2"/>
     </joint>
     <joint name="AxleLeftFront" type="continuous">

Commit message: Added Risers and Updated Origins

File: urdf/junior.urdf.xacro (robot description, xacro)
@@ -168,4 +168,23 @@
         </inertial>
     </link>
+    <!-- Risers Link -->
+    <link name="Risers">
+        <visual>
+            <geometry>
+                <mesh filename="file://$(find junior_description)/meshes/robitRiserVisual.stl"/>
+            </geometry>
+            <material name="black"/>
+        </visual>
+        <collision>
+            <geometry>
+                <mesh filename="file://$(find junior_description)/meshes/robitRiserCollision.stl"/>
+            </geometry>
+            <material name="black"/>
+        </collision>
+        <inertial>
+            <mass value="1"/>
+            <inertia ixx="0.4" ixy="0.0" ixz="0.0" iyy="0.4" iyz="0.0" izz="0.2"/>
+        </inertial>
+    </link>
     <!-- Left Front Link -->
     <link name="WheelLeftFront">
@@ -263,5 +282,5 @@
         <parent link="Chassis"/>
         <child link="BackLidarCase"/>
-        <origin xyz="-0.285 0 0.319"/>
+        <origin xyz="-0.285 0 0.339"/>
     </joint>
     <joint name="BackLidarStandJoint" type="revolute">
@@ -279,4 +298,9 @@
         <dynamics damping="0" friction="0.75"/>
         <limit lower="-1" upper="1" effort="5" velocity="2"/>
+    </joint>
+    <joint name="RisersJoint" type="fixed">
+        <parent link="Chassis"/>
+        <child link="Risers"/>
+        <origin xyz="-0.057 0 0.2655"/>
     </joint>
     <joint name="AxleLeftFront" type="continuous">
@@ -446,4 +470,14 @@
         </visual>
     </gazebo>
+    <!-- Risers -->
+    <gazebo reference="Risers">
+        <visual>
+            <material>
+                <diffuse>0.2 0.2 0.2 1</diffuse>
+                <ambient>0.1 0.1 0.1 1</ambient>
+                <emissive>0 0 0 0</emissive>
+            </material>
+        </visual>
+    </gazebo>
     <!-- WHEELS -->
     <gazebo reference="WheelLeftFront">
