Commit message: Fixed Hop-up, Still Working Towards Straightline Driving

File: urdf/junior.urdf.xacro (robot description, xacro)
@@ -31,6 +31,6 @@
         </collision>
         <inertial>
-            <mass value="35"/>
-            <inertia ixx="0.4" ixy="0.0" ixz="0.0" iyy="0.4" iyz="0.0" izz="0.2"/>
+            <mass value="45"/>
+            <inertia ixx="1.206" ixy="0.0" ixz="0.0" iyy="2.182" iyz="0.0" izz="2.182"/>
         </inertial>
     </link>
@@ -50,6 +50,6 @@
         </collision>
         <inertial>
-            <mass value="3"/>
-            <inertia ixx="0.4" ixy="0.0" ixz="0.0" iyy="0.4" iyz="0.0" izz="0.2"/>
+            <mass value="1"/>
+            <inertia ixx="0.013" ixy="0.0" ixz="0.0" iyy="0.0" iyz="0.0" izz="0.0"/>
         </inertial>
     </link>
@@ -69,6 +69,6 @@
         </collision>
         <inertial>
-            <mass value="1.5"/>
-            <inertia ixx="0.4" ixy="0.0" ixz="0.0" iyy="0.4" iyz="0.0" izz="0.2"/>
+            <mass value="1"/>
+            <inertia ixx="0.014" ixy="0.0" ixz="0.0" iyy="0.001" iyz="0.0" izz="0.001"/>
         </inertial>
     </link>
@@ -89,5 +89,5 @@
         <inertial>
             <mass value="2"/>
-            <inertia ixx="0.4" ixy="0.0" ixz="0.0" iyy="0.4" iyz="0.0" izz="0.2"/>
+            <inertia ixx="0.009" ixy="0.0" ixz="0.0" iyy="0.009" iyz="0.0" izz="0.009"/>
         </inertial>
     </link>
@@ -108,5 +108,5 @@
         <inertial>
             <mass value="0.1"/>
-            <inertia ixx="0.4" ixy="0.0" ixz="0.0" iyy="0.4" iyz="0.0" izz="0.2"/>
+            <inertia ixx="0.0" ixy="0.0" ixz="0.0" iyy="0.0" iyz="0.0" izz="0.0"/>
         </inertial>
     </link>
@@ -126,6 +126,6 @@
         </collision>
         <inertial>
-            <mass value="2"/>
-            <inertia ixx="0.4" ixy="0.0" ixz="0.0" iyy="0.4" iyz="0.0" izz="0.2"/>
+            <mass value="0.5"/>
+            <inertia ixx="0.002" ixy="0.0" ixz="0.0" iyy="0.0" iyz="0.0" izz="0.0"/>
         </inertial>
     </link>
@@ -145,6 +145,6 @@
         </collision>
         <inertial>
-            <mass value="1"/>
-            <inertia ixx="0.4" ixy="0.0" ixz="0.0" iyy="0.4" iyz="0.0" izz="0.2"/>
+            <mass value="0.5"/>
+            <inertia ixx="0.0" ixy="0.0" ixz="0.0" iyy="0.0" iyz="0.0" izz="0.0"/>
         </inertial>
     </link>
@@ -164,6 +164,6 @@
         </collision>
         <inertial>
-            <mass value="5"/>
-            <inertia ixx="0.4" ixy="0.0" ixz="0.0" iyy="0.4" iyz="0.0" izz="0.2"/>
+            <mass value="0.5"/>
+            <inertia ixx="0.0" ixy="0.0" ixz="0.0" iyy="0.0" iyz="0.0" izz="0.0"/>
         </inertial>
     </link>
@@ -183,6 +183,6 @@
         </collision>
         <inertial>
-            <mass value="1"/>
-            <inertia ixx="0.4" ixy="0.0" ixz="0.0" iyy="0.4" iyz="0.0" izz="0.2"/>
+            <mass value="0.5"/>
+            <inertia ixx="0.0" ixy="0.0" ixz="0.0" iyy="0.0" iyz="0.0" izz="0.0"/>
         </inertial>
     </link>
@@ -200,8 +200,16 @@
             </geometry>
             <material name="black"/>
-        </collision>
-        <inertial>
-            <mass value="5"/>
-            <inertia ixx="0.4" ixy="0.0" ixz="0.0" iyy="0.4" iyz="0.0" izz="0.2"/>
+            <surface>
+                <friction>
+                    <ode>
+                        <mu>0.01</mu>
+                        <mu2>0.01</mu2>
+                    </ode>
+                </friction>
+            </surface>
+        </collision>
+        <inertial>
+            <mass value="2"/>
+            <inertia ixx="0.014" ixy="0.0" ixz="0.0" iyy="0.014" iyz="0.0" izz="0.024"/>
         </inertial>
     </link>
@@ -219,8 +227,16 @@
             </geometry>
             <material name="black"/>
-        </collision>
-        <inertial>
-            <mass value="5"/>
-            <inertia ixx="0.4" ixy="0.0" ixz="0.0" iyy="0.4" iyz="0.0" izz="0.2"/>
+            <surface>
+                <friction>
+                    <ode>
+                        <mu>0.01</mu>
+                        <mu2>0.01</mu2>
+                    </ode>
+                </friction>
+            </surface>
+        </collision>
+        <inertial>
+            <mass value="2"/>
+            <inertia ixx="0.014" ixy="0.0" ixz="0.0" iyy="0.014" iyz="0.0" izz="0.024"/>
         </inertial>
     </link>
@@ -238,8 +254,16 @@
             </geometry>
             <material name="black"/>
-        </collision>
-        <inertial>
-            <mass value="5"/>
-            <inertia ixx="0.4" ixy="0.0" ixz="0.0" iyy="0.4" iyz="0.0" izz="0.2"/>
+            <surface>
+                <friction>
+                    <ode>
+                        <mu>0.01</mu>
+                        <mu2>0.01</mu2>
+                    </ode>
+                </friction>
+            </surface>
+        </collision>
+        <inertial>
+            <mass value="2"/>
+            <inertia ixx="0.014" ixy="0.0" ixz="0.0" iyy="0.014" iyz="0.0" izz="0.024"/>
         </inertial>
     </link>
@@ -257,10 +281,24 @@
             </geometry>
             <material name="black"/>
-        </collision>
-        <inertial>
-            <mass value="5"/>
-            <inertia ixx="0.4" ixy="0.0" ixz="0.0" iyy="0.4" iyz="0.0" izz="0.2"/>
-        </inertial>
-    </link>
+            <surface>
+                <friction>
+                    <ode>
+                        <mu>0.01</mu>
+                        <mu2>0.01</mu2>
+                    </ode>
+                </friction>
+            </surface>
+        </collision>
+        <inertial>
+            <mass value="2"/>
+            <inertia ixx="0.014" ixy="0.0" ixz="0.0" iyy="0.014" iyz="0.0" izz="0.024"/>
+        </inertial>
+    </link>
+    <!-- Graveyard of Wheel Inertias
+    Ted v1 : <inertia ixx="0.007" ixy="0.0" ixz="0.0" iyy="0.014" iyz="0.0" izz="0.007"/>
+    Cylinder Math : <inertia ixx="0.014" ixy="0.0" ixz="0.0" iyy="0.014" iyz="0.0" izz="0.024"/>
+    Box Math : <inertia ixx="0.0183" ixy="0.0" ixz="0.0" iyy="0.033" iyz="0.0" izz="0.033"/>
+    Logi v1 : <inertia ixx="0.014" ixy="0.0" ixz="0.0" iyy="0.04" iyz="0.0" izz="0.024"/>
+    -->
     <!-- START OF JOINTS -->
     <joint name="ChassisJoint" type="fixed">
@@ -528,7 +566,7 @@
             <!-- kinematics -->
             <wheel_separation>0.52</wheel_separation>
-            <wheel_diameter>0.105</wheel_diameter>
+            <wheel_diameter>0.315</wheel_diameter>
             <!-- Limits -->
-            <max_wheel_torque>200.0</max_wheel_torque>
+            <max_wheel_torque>40.0</max_wheel_torque>
             <max_wheel_acceleration>10.0</max_wheel_acceleration>
             <!-- Output -->

Commit message: Made Inertial Origin Changes

File: urdf/junior.urdf.xacro (robot description, xacro)
@@ -212,4 +212,5 @@
             <mass value="2"/>
             <inertia ixx="0.014" ixy="0.0" ixz="0.0" iyy="0.014" iyz="0.0" izz="0.024"/>
+            <origin xyz="0 0 0" rpy="1.57 0 0"/>
         </inertial>
     </link>
@@ -239,4 +240,5 @@
             <mass value="2"/>
             <inertia ixx="0.014" ixy="0.0" ixz="0.0" iyy="0.014" iyz="0.0" izz="0.024"/>
+            <origin xyz="0 0 0" rpy="1.57 0 0"/>
         </inertial>
     </link>
@@ -266,4 +268,5 @@
             <mass value="2"/>
             <inertia ixx="0.014" ixy="0.0" ixz="0.0" iyy="0.014" iyz="0.0" izz="0.024"/>
+            <origin xyz="0 0 0" rpy="1.57 0 0"/>
         </inertial>
     </link>
@@ -293,4 +296,5 @@
             <mass value="2"/>
             <inertia ixx="0.014" ixy="0.0" ixz="0.0" iyy="0.014" iyz="0.0" izz="0.024"/>
+            <origin xyz="0 0 0" rpy="1.57 0 0"/>
         </inertial>
     </link>
@@ -565,9 +569,9 @@
             <right_joint>AxleRightBack</right_joint>
             <!-- kinematics -->
-            <wheel_separation>0.52</wheel_separation>
+            <wheel_separation>0.435</wheel_separation>
             <wheel_diameter>0.315</wheel_diameter>
             <!-- Limits -->
             <max_wheel_torque>40.0</max_wheel_torque>
-            <max_wheel_acceleration>10.0</max_wheel_acceleration>
+            <max_wheel_acceleration>5.0</max_wheel_acceleration>
             <!-- Output -->
             <odometry_frame>odom</odometry_frame>

Commit message: Updated Chassis Visual Further

File: urdf/junior.urdf.xacro (robot description, xacro)
@@ -20,7 +20,6 @@
         <visual>
             <geometry>
-                <mesh filename="file://$(find junior_description)/meshes/robitChassisVisual.stl"/>
-            </geometry>
-            <material name="red"/>
+                <mesh filename="file://$(find junior_description)/meshes/robitChassisVisual.dae"/>
+            </geometry>
         </visual>
         <collision>
@@ -384,11 +383,4 @@
     <!-- Chassis -->
     <gazebo reference="Chassis">
-        <visual>
-            <material>
-                <diffuse>1 0 0 1</diffuse>
-                <ambient>0.4 0.05 0.05 1</ambient>
-                <emissive>0 0 0 0</emissive>
-            </material>
-        </visual>
     </gazebo>
     <!-- Front Bumper -->

Commit message: Working Forward Drive and Turning, Reversing Still Deviates

File: urdf/junior.urdf.xacro (robot description, xacro)
@@ -196,12 +196,16 @@
         <collision>
             <geometry>
-                <mesh filename="file://$(find junior_description)/meshes/robitWheel.stl"/>
-            </geometry>
+                <mesh filename="file://$(find junior_description)/meshes/robitWheelCollision.dae"/>
+            </geometry>
+            <!-- <origin xyz="0 0 0" rpy="1.57 0 0"/> -->
             <material name="black"/>
             <surface>
                 <friction>
                     <ode>
-                        <mu>0.01</mu>
-                        <mu2>0.01</mu2>
+                        <mu>1.0</mu>
+                        <mu2>1.0</mu2>
+                        <kp>10000000.0</kp>
+                        <kd>1.0</kd>
+                        <fdir>1 0 0</fdir>
                     </ode>
                 </friction>
@@ -210,5 +214,5 @@
         <inertial>
             <mass value="2"/>
-            <inertia ixx="0.014" ixy="0.0" ixz="0.0" iyy="0.014" iyz="0.0" izz="0.024"/>
+            <inertia ixx="0.014240625" ixy="0.0" ixz="0.0" iyy="0.014240625" iyz="0.0" izz="0.02480625"/>
             <origin xyz="0 0 0" rpy="1.57 0 0"/>
         </inertial>
@@ -224,12 +228,16 @@
         <collision>
             <geometry>
-                <mesh filename="file://$(find junior_description)/meshes/robitWheel.stl"/>
-            </geometry>
+                <mesh filename="file://$(find junior_description)/meshes/robitWheelCollision.dae"/>
+            </geometry>
+            <!-- <origin xyz="0 0 0" rpy="1.57 0 0"/> -->
             <material name="black"/>
             <surface>
                 <friction>
                     <ode>
-                        <mu>0.01</mu>
-                        <mu2>0.01</mu2>
+                        <mu>1.0</mu>
+                        <mu2>1.0</mu2>
+                        <kp>10000000.0</kp>
+                        <kd>1.0</kd>
+                        <fdir>1 0 0</fdir>
                     </ode>
                 </friction>
@@ -238,5 +246,5 @@
         <inertial>
             <mass value="2"/>
-            <inertia ixx="0.014" ixy="0.0" ixz="0.0" iyy="0.014" iyz="0.0" izz="0.024"/>
+            <inertia ixx="0.014240625" ixy="0.0" ixz="0.0" iyy="0.014240625" iyz="0.0" izz="0.02480625"/>
             <origin xyz="0 0 0" rpy="1.57 0 0"/>
         </inertial>
@@ -252,12 +260,16 @@
         <collision>
             <geometry>
-                <mesh filename="file://$(find junior_description)/meshes/robitWheel.stl"/>
-            </geometry>
+                <mesh filename="file://$(find junior_description)/meshes/robitWheelCollision.dae"/>
+            </geometry>
+            <!-- <origin xyz="0 0 0" rpy="1.57 0 0"/> -->
             <material name="black"/>
             <surface>
                 <friction>
                     <ode>
-                        <mu>0.01</mu>
-                        <mu2>0.01</mu2>
+                        <mu>1.0</mu>
+                        <mu2>1.0</mu2>
+                        <kp>10000000.0</kp>
+                        <kd>1.0</kd>
+                        <fdir>1 0 0</fdir>
                     </ode>
                 </friction>
@@ -266,5 +278,5 @@
         <inertial>
             <mass value="2"/>
-            <inertia ixx="0.014" ixy="0.0" ixz="0.0" iyy="0.014" iyz="0.0" izz="0.024"/>
+            <inertia ixx="0.014240625" ixy="0.0" ixz="0.0" iyy="0.014240625" iyz="0.0" izz="0.02480625"/>
             <origin xyz="0 0 0" rpy="1.57 0 0"/>
         </inertial>
@@ -280,12 +292,16 @@
         <collision>
             <geometry>
-                <mesh filename="file://$(find junior_description)/meshes/robitWheel.stl"/>
-            </geometry>
+                <mesh filename="file://$(find junior_description)/meshes/robitWheelCollision.dae"/>
+            </geometry>
+            <!-- <origin xyz="0 0 0" rpy="1.57 0 0"/> -->
             <material name="black"/>
             <surface>
                 <friction>
                     <ode>
-                        <mu>0.01</mu>
-                        <mu2>0.01</mu2>
+                        <mu>1.0</mu>
+                        <mu2>1.0</mu2>
+                        <kp>10000000.0</kp>
+                        <kd>1.0</kd>
+                        <fdir>1 0 0</fdir>
                     </ode>
                 </friction>
@@ -294,5 +310,5 @@
         <inertial>
             <mass value="2"/>
-            <inertia ixx="0.014" ixy="0.0" ixz="0.0" iyy="0.014" iyz="0.0" izz="0.024"/>
+            <inertia ixx="0.014240625" ixy="0.0" ixz="0.0" iyy="0.014240625" iyz="0.0" izz="0.02480625"/>
             <origin xyz="0 0 0" rpy="1.57 0 0"/>
         </inertial>
@@ -303,4 +319,5 @@
     Box Math : <inertia ixx="0.0183" ixy="0.0" ixz="0.0" iyy="0.033" iyz="0.0" izz="0.033"/>
     Logi v1 : <inertia ixx="0.014" ixy="0.0" ixz="0.0" iyy="0.04" iyz="0.0" izz="0.024"/>
+    CURRENT: Precision Cylinder : <inertia ixx="0.014240625" ixy="0.0" ixz="0.0" iyy="0.014240625" iyz="0.0" izz="0.02480625"/>
     -->
     <!-- START OF JOINTS -->
@@ -564,6 +581,6 @@
             <wheel_diameter>0.315</wheel_diameter>
             <!-- Limits -->
-            <max_wheel_torque>40.0</max_wheel_torque>
-            <max_wheel_acceleration>5.0</max_wheel_acceleration>
+            <max_wheel_torque>30.0</max_wheel_torque>
+            <max_wheel_acceleration>3.0</max_wheel_acceleration>
             <!-- Output -->
             <odometry_frame>odom</odometry_frame>
