Commit message: Back Lidar --> Back Camera

File: urdf/junior.urdf.xacro (robot description, xacro)
@@ -110,15 +110,15 @@
         </inertial>
     </link>
-    <!-- Back Lidar Case Link -->
-    <link name="BackLidarCase">
-        <visual>
-            <geometry>
-                <mesh filename="file://$(find junior_description)/meshes/robitBackLidarCase.stl"/>
-            </geometry>
-            <material name="black"/>
-        </visual>
-        <collision>
-            <geometry>
-                <mesh filename="file://$(find junior_description)/meshes/robitBackLidarCase.stl"/>
+    <!-- Back Camera Case Link -->
+    <link name="BackCameraCase">
+        <visual>
+            <geometry>
+                <mesh filename="file://$(find junior_description)/meshes/robitBackCameraCase.stl"/>
+            </geometry>
+            <material name="black"/>
+        </visual>
+        <collision>
+            <geometry>
+                <mesh filename="file://$(find junior_description)/meshes/robitBackCameraCase.stl"/>
             </geometry>
             <material name="black"/>
@@ -129,9 +129,9 @@
         </inertial>
     </link>
-    <!-- Back Lidar Stand Link -->
-    <link name="BackLidarStand">
-        <visual>
-            <geometry>
-                <mesh filename="file://$(find junior_description)/meshes/robitBackLidarStand.stl"/>
+    <!-- Back Camera Stand Link -->
+    <link name="BackCameraStand">
+        <visual>
+            <geometry>
+                <mesh filename="file://$(find junior_description)/meshes/robitBackCameraStand.stl"/>
             </geometry>
             <material name="silver"/>
@@ -139,5 +139,5 @@
         <collision>
             <geometry>
-                <mesh filename="file://$(find junior_description)/meshes/robitBackLidarStand.stl"/>
+                <mesh filename="file://$(find junior_description)/meshes/robitBackCameraStand.stl"/>
             </geometry>
             <material name="silver"/>
@@ -148,9 +148,9 @@
         </inertial>
     </link>
-    <!-- Back Lidar Head -->
-    <link name="BackLidarHead">
-        <visual>
-            <geometry>
-                <mesh filename="file://$(find junior_description)/meshes/robitBackLidarHead.stl"/>
+    <!-- Back Camera Head Link -->
+    <link name="BackCameraHead">
+        <visual>
+            <geometry>
+                <mesh filename="file://$(find junior_description)/meshes/robitBackCameraHead.stl"/>
             </geometry>
             <material name="silver"/>
@@ -158,5 +158,5 @@
         <collision>
             <geometry>
-                <mesh filename="file://$(find junior_description)/meshes/robitBackLidarHead.stl"/>
+                <mesh filename="file://$(find junior_description)/meshes/robitBackCameraHead.stl"/>
             </geometry>
             <material name="silver"/>
@@ -196,7 +196,8 @@
         <collision>
             <geometry>
-                <mesh filename="file://$(find junior_description)/meshes/robitWheelCollision.dae"/>
-            </geometry>
-            <!-- <origin xyz="0 0 0" rpy="1.57 0 0"/> -->
+                <!-- <mesh filename="file://$(find junior_description)/meshes/robitWheelCollision.dae"/> -->
+                <cylinder length="0.105" radius="0.1575"/>
+            </geometry>
+            <origin xyz="0 0 0" rpy="1.57079632679 0 0"/>
             <material name="black"/>
             <surface>
@@ -215,5 +216,5 @@
             <mass value="2"/>
             <inertia ixx="0.014240625" ixy="0.0" ixz="0.0" iyy="0.014240625" iyz="0.0" izz="0.02480625"/>
-            <origin xyz="0 0 0" rpy="1.57 0 0"/>
+            <origin xyz="0 0 0" rpy="1.57079632679 0 0"/>
         </inertial>
     </link>
@@ -228,7 +229,8 @@
         <collision>
             <geometry>
-                <mesh filename="file://$(find junior_description)/meshes/robitWheelCollision.dae"/>
-            </geometry>
-            <!-- <origin xyz="0 0 0" rpy="1.57 0 0"/> -->
+                <!-- <mesh filename="file://$(find junior_description)/meshes/robitWheelCollision.dae"/> -->
+                <cylinder length="0.105" radius="0.1575"/>
+            </geometry>
+            <origin xyz="0 0 0" rpy="1.57079632679 0 0"/>
             <material name="black"/>
             <surface>
@@ -247,5 +249,5 @@
             <mass value="2"/>
             <inertia ixx="0.014240625" ixy="0.0" ixz="0.0" iyy="0.014240625" iyz="0.0" izz="0.02480625"/>
-            <origin xyz="0 0 0" rpy="1.57 0 0"/>
+            <origin xyz="0 0 0" rpy="1.57079632679 0 0"/>
         </inertial>
     </link>
@@ -260,7 +262,8 @@
         <collision>
             <geometry>
-                <mesh filename="file://$(find junior_description)/meshes/robitWheelCollision.dae"/>
-            </geometry>
-            <!-- <origin xyz="0 0 0" rpy="1.57 0 0"/> -->
+                <!-- <mesh filename="file://$(find junior_description)/meshes/robitWheelCollision.dae"/> -->
+                <cylinder length="0.105" radius="0.1575"/>
+            </geometry>
+            <origin xyz="0 0 0" rpy="1.57079632679 0 0"/>
             <material name="black"/>
             <surface>
@@ -279,5 +282,5 @@
             <mass value="2"/>
             <inertia ixx="0.014240625" ixy="0.0" ixz="0.0" iyy="0.014240625" iyz="0.0" izz="0.02480625"/>
-            <origin xyz="0 0 0" rpy="1.57 0 0"/>
+            <origin xyz="0 0 0" rpy="1.57079632679 0 0"/>
         </inertial>
     </link>
@@ -292,7 +295,8 @@
         <collision>
             <geometry>
-                <mesh filename="file://$(find junior_description)/meshes/robitWheelCollision.dae"/>
-            </geometry>
-            <!-- <origin xyz="0 0 0" rpy="1.57 0 0"/> -->
+                <!-- <mesh filename="file://$(find junior_description)/meshes/robitWheelCollision.dae"/> -->
+                <cylinder length="0.105" radius="0.1575"/>
+            </geometry>
+            <origin xyz="0 0 0" rpy="1.57079632679 0 0"/>
             <material name="black"/>
             <surface>
@@ -311,5 +315,5 @@
             <mass value="2"/>
             <inertia ixx="0.014240625" ixy="0.0" ixz="0.0" iyy="0.014240625" iyz="0.0" izz="0.02480625"/>
-            <origin xyz="0 0 0" rpy="1.57 0 0"/>
+            <origin xyz="0 0 0" rpy="1.57079632679 0 0"/>
         </inertial>
     </link>
@@ -320,4 +324,5 @@
     Logi v1 : <inertia ixx="0.014" ixy="0.0" ixz="0.0" iyy="0.04" iyz="0.0" izz="0.024"/>
     CURRENT: Precision Cylinder : <inertia ixx="0.014240625" ixy="0.0" ixz="0.0" iyy="0.014240625" iyz="0.0" izz="0.02480625"/>
+    Gazebo Cylinder : <inertia ixx="0.15" ixy="0.0" ixz="0.0" iyy="0.15" iyz="0.0" izz="0.13"/>
     -->
     <!-- START OF JOINTS -->
@@ -337,23 +342,23 @@
         <origin xyz="0.075 0 0"/>
     </joint>
-    <joint name="BackLidarHolster" type="fixed">
-        <parent link="Chassis"/>
-        <child link="BackLidarCase"/>
+    <joint name="BackCameraHolster" type="fixed">
+        <parent link="Chassis"/>
+        <child link="BackCameraCase"/>
         <origin xyz="-0.285 0 0.339"/>
     </joint>
-    <joint name="BackLidarStandJoint" type="revolute">
-        <parent link="BackLidarCase"/>
-        <child link="BackLidarStand"/>
+    <joint name="BackCameraStandJoint" type="fixed">
+        <parent link="BackCameraCase"/>
+        <child link="BackCameraStand"/>
         <origin xyz="0 0 -0.045"/>
         <axis xyz="0 0 1"/>
-        <limit lower="-1" upper="1" effort="5" velocity="2"/>
-    </joint>
-    <joint name="BackLidarHeadJoint" type="revolute">
-        <parent link="BackLidarStand"/>
-        <child link="BackLidarHead"/>
+        <!-- <limit lower="-1" upper="1" effort="5" velocity="2"/>  FOR REVOLUTE -->
+    </joint>
+    <joint name="BackCameraHeadJoint" type="fixed">
+        <parent link="BackCameraStand"/>
+        <child link="BackCameraHead"/>
         <origin xyz="0 0 0.05" rpy="0 -3.14 0"/>
         <axis xyz="0 1 0"/>
-        <dynamics damping="0" friction="0.75"/>
-        <limit lower="-1" upper="1" effort="5" velocity="2"/>
+        <!-- <dynamics damping="0" friction="0.75"/>
+        <limit lower="-1" upper="1" effort="5" velocity="2"/> FOR REVOLUTE -->
     </joint>
     <joint name="RisersJoint" type="fixed">
@@ -466,6 +471,6 @@
         </visual>
     </gazebo>
-    <!-- Back Lidar Case -->
-    <gazebo reference="BackLidarCase">
+    <!-- Back Camera Case -->
+    <gazebo reference="BackCameraCase">
         <visual>
             <material>
@@ -477,5 +482,5 @@
     </gazebo>
     <!-- Back Lidar Stand -->
-    <gazebo reference="BackLidarStand">
+    <gazebo reference="BackCameraStand">
         <visual>
             <material>
@@ -487,5 +492,5 @@
     </gazebo>
     <!-- Back Lidar Head -->
-    <gazebo reference="BackLidarHead">
+    <gazebo reference="BackCameraHead">
         <sensor name="blaser" type="ray">
             <pose> 0 0 0 0 0 </pose>
@@ -510,5 +515,5 @@
                 </ros>
                 <output_type>sensor_msgs/LaserScan</output_type>
-                <frame_name>BackLidarHead</frame_name>
+                <frame_name>BackCameraHead</frame_name>
             </plugin>
         </sensor>

Commit message: Implemented Actual Back Lidar

File: urdf/junior.urdf.xacro (robot description, xacro)
@@ -186,4 +186,30 @@
         </inertial>
     </link>
+    <!-- Back Lidar Link -->
+    <link name="BackLidar">
+        <visual>
+            <geometry>
+                <mesh filename="file://$(find junior_description)/meshes/hokuyo_urg_04lx.dae"/>
+            </geometry>
+            <material name="black"/>
+        </visual>
+        <collision>
+            <geometry>
+                <mesh filename="file://$(find junior_description)/meshes/hokuyo_urg_04lx.dae"/>
+            </geometry>
+            <material name="black"/>
+        </collision>
+        <inertial>
+            <mass value="0.2"/>
+            <inertia ixx="0.0" ixy="0.0" ixz="0.0" iyy="0.0" iyz="0.0" izz="0.0"/>
+        </inertial>
+    </link>
+    <!-- Back Lidar Scanner Link -->
+    <link name="BackLidarScanner">
+        <inertial>
+            <mass value="0.001"/>
+            <inertia ixx="0.0" ixy="0.0" ixz="0.0" iyy="0.0" iyz="0.0" izz="0.0"/>
+        </inertial>
+    </link>
     <!-- Left Front Link -->
     <link name="WheelLeftFront">
@@ -196,8 +222,8 @@
         <collision>
             <geometry>
-                <!-- <mesh filename="file://$(find junior_description)/meshes/robitWheelCollision.dae"/> -->
-                <cylinder length="0.105" radius="0.1575"/>
-            </geometry>
-            <origin xyz="0 0 0" rpy="1.57079632679 0 0"/>
+                <mesh filename="file://$(find junior_description)/meshes/robitWheelCollision.dae"/>
+                <!-- <cylinder length="0.105" radius="0.1575"/> -->
+            </geometry>
+            <!-- <origin xyz="0 0 0" rpy="1.57079632679 0 0"/> -->
             <material name="black"/>
             <surface>
@@ -229,8 +255,8 @@
         <collision>
             <geometry>
-                <!-- <mesh filename="file://$(find junior_description)/meshes/robitWheelCollision.dae"/> -->
-                <cylinder length="0.105" radius="0.1575"/>
-            </geometry>
-            <origin xyz="0 0 0" rpy="1.57079632679 0 0"/>
+                <mesh filename="file://$(find junior_description)/meshes/robitWheelCollision.dae"/>
+                <!-- <cylinder length="0.105" radius="0.1575"/> -->
+            </geometry>
+            <!-- <origin xyz="0 0 0" rpy="1.57079632679 0 0"/> -->
             <material name="black"/>
             <surface>
@@ -262,8 +288,8 @@
         <collision>
             <geometry>
-                <!-- <mesh filename="file://$(find junior_description)/meshes/robitWheelCollision.dae"/> -->
-                <cylinder length="0.105" radius="0.1575"/>
-            </geometry>
-            <origin xyz="0 0 0" rpy="1.57079632679 0 0"/>
+                <mesh filename="file://$(find junior_description)/meshes/robitWheelCollision.dae"/>
+                <!-- <cylinder length="0.105" radius="0.1575"/> -->
+            </geometry>
+            <!-- <origin xyz="0 0 0" rpy="1.57079632679 0 0"/> -->
             <material name="black"/>
             <surface>
@@ -295,8 +321,8 @@
         <collision>
             <geometry>
-                <!-- <mesh filename="file://$(find junior_description)/meshes/robitWheelCollision.dae"/> -->
-                <cylinder length="0.105" radius="0.1575"/>
-            </geometry>
-            <origin xyz="0 0 0" rpy="1.57079632679 0 0"/>
+                <mesh filename="file://$(find junior_description)/meshes/robitWheelCollision.dae"/>
+                <!-- <cylinder length="0.105" radius="0.1575"/> -->
+            </geometry>
+            <!-- <origin xyz="0 0 0" rpy="1.57079632679 0 0"/> -->
             <material name="black"/>
             <surface>
@@ -367,4 +393,14 @@
         <origin xyz="-0.057 0 0.2655"/>
     </joint>
+    <joint name="BackLidarJoint" type="fixed">
+        <parent link="BackCameraCase"/>
+        <child link="BackLidar"/>
+        <origin xyz="0 0 0.045" rpy="0 0 -3.14"/>
+    </joint>
+    <joint name="BackLidarScannerJoint" type="fixed">
+        <parent link="BackLidar"/>
+        <child link="BackLidarScanner"/>
+        <origin xyz="0 0 0.03" rpy="0 0 0"/>
+    </joint>
     <joint name="AxleLeftFront" type="continuous">
         <parent link="Chassis"/>
@@ -440,5 +476,5 @@
         <sensor name="laser" type="ray">
             <pose> 0 0 0 0 0 0 </pose>
-            <visualize>true</visualize>
+            <visualize>false</visualize> <!-- TURN TO TRUE WHEN TESTING THE LIDAR -->
             <update_rate>10</update_rate>
             <ray>
@@ -493,46 +529,59 @@
     <!-- Back Lidar Head -->
     <gazebo reference="BackCameraHead">
+        <visual>
+            <material>
+                <diffuse>0.77 0.78 0.78 1</diffuse>
+                <ambient>0.385 0.39 0.39 1</ambient>
+                <emissive>0 0 0 0</emissive>
+            </material>
+        </visual>
+    </gazebo>
+    <!-- Risers -->
+    <gazebo reference="Risers">
+        <visual>
+            <material>
+                <diffuse>0.2 0.2 0.2 1</diffuse>
+                <ambient>0.1 0.1 0.1 1</ambient>
+                <emissive>0 0 0 0</emissive>
+            </material>
+        </visual>
+    </gazebo>
+    <!-- Back Lidar -->
+    <gazebo reference="BackLidar">
+    </gazebo>
+    <!-- Back Lidar Scanner -->
+    <gazebo reference="BackLidarScanner">
         <sensor name="blaser" type="ray">
-            <pose> 0 0 0 0 0 </pose>
-            <visualize>true</visualize>
+            <pose>0 0 0 0 0 0</pose>
+            <visualize>false</visualize> <!-- TURN TO TRUE WHEN TESTING THE LIDAR -->
             <update_rate>10</update_rate>
             <ray>
                 <scan>
                     <horizontal>
-                    <samples>120</samples>
-                    <min_angle>-0.52</min_angle>
-                    <max_angle>0.52</max_angle>
+                        <samples>640</samples>
+                        <resolution>1</resolution>
+                        <min_angle>-2.3561</min_angle>
+                        <max_angle>2.3561</max_angle>
                     </horizontal>
                 </scan>
                 <range>
-                    <min>0.1</min>
-                    <max>2</max>
+                    <min>0.035</min> <!-- Was 0.02 -->
+                    <max>4.0</max>
+                    <resolution>0.00628318531</resolution>
                 </range>
+                <noise>
+                    <type>gaussian</type>
+                    <mean>0.0</mean>
+                    <stddev>0.01</stddev>
+                </noise>
             </ray>
-            <plugin name="bl_controller" filename="libgazebo_ros_ray_sensor.so">
+			<plugin name="bl_controller" filename="libgazebo_ros_ray_sensor.so">
                 <ros>
                     <argument>-/out:=scan</argument>
                 </ros>
-                <output_type>sensor_msgs/LaserScan</output_type>
-                <frame_name>BackCameraHead</frame_name>
-            </plugin>
-        </sensor>
-        <visual>
-            <material>
-                <diffuse>0.77 0.78 0.78 1</diffuse>
-                <ambient>0.385 0.39 0.39 1</ambient>
-                <emissive>0 0 0 0</emissive>
-            </material>
-        </visual>
-    </gazebo>
-    <!-- Risers -->
-    <gazebo reference="Risers">
-        <visual>
-            <material>
-                <diffuse>0.2 0.2 0.2 1</diffuse>
-                <ambient>0.1 0.1 0.1 1</ambient>
-                <emissive>0 0 0 0</emissive>
-            </material>
-        </visual>
+				<output_type>sensor_msgs/LaserScan</output_type>
+                <frame_name>BackLidar</frame_name>
+			</plugin>
+		</sensor>
     </gazebo>
     <!-- WHEELS -->
