Commit message: Minor Changes to Drive Plugin, Reverse Still Broken

File: urdf/junior.urdf.xacro (robot description, xacro)
@@ -26,4 +26,5 @@
             <geometry>
                 <mesh filename="file://$(find junior_description)/meshes/robitChassis.stl"/>
+               <!-- <box size="0.642 0.39 0.412"/> -->
             </geometry>
             <material name="red"/>
@@ -31,5 +32,5 @@
         <inertial>
             <mass value="45"/>
-            <inertia ixx="1.206" ixy="0.0" ixz="0.0" iyy="2.182" iyz="0.0" izz="2.182"/>
+            <inertia ixx="1.20932883" ixy="0.0" ixz="0.0" iyy="2.18651931" iyz="0.0" izz="2.18651931"/>
         </inertial>
     </link>
@@ -49,6 +50,6 @@
         </collision>
         <inertial>
-            <mass value="1"/>
-            <inertia ixx="0.013" ixy="0.0" ixz="0.0" iyy="0.0" iyz="0.0" izz="0.0"/>
+            <mass value="0.01"/>
+            <inertia ixx="0.0" ixy="0.0" ixz="0.0" iyy="0.0" iyz="0.0" izz="0.0"/>
         </inertial>
     </link>
@@ -68,6 +69,6 @@
         </collision>
         <inertial>
-            <mass value="1"/>
-            <inertia ixx="0.014" ixy="0.0" ixz="0.0" iyy="0.001" iyz="0.0" izz="0.001"/>
+            <mass value="0.01"/>
+            <inertia ixx="0.0" ixy="0.0" ixz="0.0" iyy="0.0" iyz="0.0" izz="0.0"/>
         </inertial>
     </link>
@@ -87,6 +88,6 @@
         </collision>
         <inertial>
-            <mass value="2"/>
-            <inertia ixx="0.009" ixy="0.0" ixz="0.0" iyy="0.009" iyz="0.0" izz="0.009"/>
+            <mass value="0.01"/>
+            <inertia ixx="0.0" ixy="0.0" ixz="0.0" iyy="0.0" iyz="0.0" izz="0.0"/>
         </inertial>
     </link>
@@ -106,5 +107,5 @@
         </collision>
         <inertial>
-            <mass value="0.1"/>
+            <mass value="0.01"/>
             <inertia ixx="0.0" ixy="0.0" ixz="0.0" iyy="0.0" iyz="0.0" izz="0.0"/>
         </inertial>
@@ -125,6 +126,6 @@
         </collision>
         <inertial>
-            <mass value="0.5"/>
-            <inertia ixx="0.002" ixy="0.0" ixz="0.0" iyy="0.0" iyz="0.0" izz="0.0"/>
+            <mass value="0.01"/>
+            <inertia ixx="0.0" ixy="0.0" ixz="0.0" iyy="0.0" iyz="0.0" izz="0.0"/>
         </inertial>
     </link>
@@ -144,5 +145,5 @@
         </collision>
         <inertial>
-            <mass value="0.5"/>
+            <mass value="0.01"/>
             <inertia ixx="0.0" ixy="0.0" ixz="0.0" iyy="0.0" iyz="0.0" izz="0.0"/>
         </inertial>
@@ -163,5 +164,5 @@
         </collision>
         <inertial>
-            <mass value="0.5"/>
+            <mass value="0.01"/>
             <inertia ixx="0.0" ixy="0.0" ixz="0.0" iyy="0.0" iyz="0.0" izz="0.0"/>
         </inertial>
@@ -182,5 +183,5 @@
         </collision>
         <inertial>
-            <mass value="0.5"/>
+            <mass value="0.01"/>
             <inertia ixx="0.0" ixy="0.0" ixz="0.0" iyy="0.0" iyz="0.0" izz="0.0"/>
         </inertial>
@@ -201,5 +202,5 @@
         </collision>
         <inertial>
-            <mass value="0.2"/>
+            <mass value="0.01"/>
             <inertia ixx="0.0" ixy="0.0" ixz="0.0" iyy="0.0" iyz="0.0" izz="0.0"/>
         </inertial>
@@ -217,6 +218,8 @@
             <geometry>
                 <mesh filename="file://$(find junior_description)/meshes/robitWheel.stl"/>
-            </geometry>
-            <material name="black"/>
+                <!-- <cylinder length="0.105" radius="0.1575"/> -->
+            </geometry>
+            <material name="black"/>
+            <!-- <origin xyz="0 0 0" rpy="1.57079632679 0 0"/>  Comment Out for Mesh -->
         </visual>
         <collision>
@@ -230,7 +233,7 @@
                 <friction>
                     <ode>
-                        <mu>1.0</mu>
-                        <mu2>1.0</mu2>
-                        <kp>10000000.0</kp>
+                        <mu>0.7</mu>
+                        <mu2>0.7</mu2>
+                        <kp>1000000</kp>
                         <kd>1.0</kd>
                         <fdir>1 0 0</fdir>
@@ -250,6 +253,8 @@
             <geometry>
                 <mesh filename="file://$(find junior_description)/meshes/robitWheel.stl"/>
-            </geometry>
-            <material name="black"/>
+                <!-- <cylinder length="0.105" radius="0.1575"/> -->
+            </geometry>
+            <material name="black"/>
+            <!-- <origin xyz="0 0 0" rpy="1.57079632679 0 0"/>  Comment Out for Mesh -->
         </visual>
         <collision>
@@ -263,7 +268,7 @@
                 <friction>
                     <ode>
-                        <mu>1.0</mu>
-                        <mu2>1.0</mu2>
-                        <kp>10000000.0</kp>
+                        <mu>0.7</mu>
+                        <mu2>0.7</mu2>
+                        <kp>1000000</kp>
                         <kd>1.0</kd>
                         <fdir>1 0 0</fdir>
@@ -283,6 +288,8 @@
             <geometry>
                 <mesh filename="file://$(find junior_description)/meshes/robitWheel.stl"/>
-            </geometry>
-            <material name="black"/>
+                <!-- <cylinder length="0.105" radius="0.1575"/> -->
+            </geometry>
+            <material name="black"/>
+            <!-- <origin xyz="0 0 0" rpy="1.57079632679 0 0"/>  Comment Out for Mesh -->
         </visual>
         <collision>
@@ -296,7 +303,7 @@
                 <friction>
                     <ode>
-                        <mu>1.0</mu>
-                        <mu2>1.0</mu2>
-                        <kp>10000000.0</kp>
+                        <mu>0.7</mu>
+                        <mu2>0.7</mu2>
+                        <kp>1000000</kp>
                         <kd>1.0</kd>
                         <fdir>1 0 0</fdir>
@@ -316,6 +323,8 @@
             <geometry>
                 <mesh filename="file://$(find junior_description)/meshes/robitWheel.stl"/>
-            </geometry>
-            <material name="black"/>
+                <!-- <cylinder length="0.105" radius="0.1575"/> -->
+            </geometry>
+            <material name="black"/>
+            <!-- <origin xyz="0 0 0" rpy="1.57079632679 0 0"/>  Comment Out for Mesh -->
         </visual>
         <collision>
@@ -329,7 +338,7 @@
                 <friction>
                     <ode>
-                        <mu>1.0</mu>
-                        <mu2>1.0</mu2>
-                        <kp>10000000.0</kp>
+                        <mu>0.7</mu>
+                        <mu2>0.7</mu2>
+                        <kp>1000000</kp>
                         <kd>1.0</kd>
                         <fdir>1 0 0</fdir>
@@ -624,6 +633,5 @@
     <!-- END OF WHEELS -->
     <gazebo>
-        <plugin name="wheel_drive_controller" filename="libgazebo_ros_diff_drive.so">
-            <!-- wheels -->
+        <plugin name="diff_drive_controller" filename="libgazebo_ros_diff_drive.so">
             <num_wheel_pairs>2</num_wheel_pairs>
             <left_joint>AxleLeftFront</left_joint>
@@ -631,22 +639,20 @@
             <right_joint>AxleRightFront</right_joint>
             <right_joint>AxleRightBack</right_joint>
-            <!-- kinematics -->
             <wheel_separation>0.435</wheel_separation>
             <wheel_diameter>0.315</wheel_diameter>
-            <!-- Limits -->
             <max_wheel_torque>30.0</max_wheel_torque>
-            <max_wheel_acceleration>3.0</max_wheel_acceleration>
-            <!-- Output -->
+            <max_wheel_acceleration>0.7</max_wheel_acceleration>
+            <!-- Max Teleop Speeds
+                Forward Speed: 1.8 m/s
+                Reverse Speed: 0 m/s
+                Left Turn Speed: 7 m/s
+                Right Turn Speed: 7 m/s
+            -->
             <odometry_frame>odom</odometry_frame>
             <robot_base_frame>base_link</robot_base_frame>
-            <!-- topic & re remappings -->
-            <!-- ros>
-                <namespace>/</namespace>
-                <argument>/cmd_vel:=cmd_vel</argument>
-                <argument>/odom:=odom</argument>
-            </ros -->
             <publish_odom>true</publish_odom>
             <publish_odom_tf>true</publish_odom_tf>
-            <update_rate>30.0</update_rate>
+            <publish_wheel_tf>true</publish_wheel_tf>
+            <update_rate>100.0</update_rate>
         </plugin>
     </gazebo>

Commit message: Big Visual and Link Changes to Chassis and Wheels

File: urdf/junior.urdf.xacro (robot description, xacro)
@@ -25,5 +25,5 @@
         <collision>
             <geometry>
-                <mesh filename="file://$(find junior_description)/meshes/robitChassis.stl"/>
+                <mesh filename="file://$(find junior_description)/meshes/robitChassisCollision.dae"/>
                <!-- <box size="0.642 0.39 0.412"/> -->
             </geometry>
@@ -35,42 +35,4 @@
         </inertial>
     </link>
-    <!-- Front Bumper Link -->
-    <link name="FrontBumper">
-        <visual>
-            <geometry>
-                <mesh filename="file://$(find junior_description)/meshes/robitFrontBumper.stl"/>
-            </geometry>
-            <material name="black"/>
-        </visual>
-        <collision>
-            <geometry>
-                <mesh filename="file://$(find junior_description)/meshes/robitFrontBumper.stl"/>
-            </geometry>
-            <material name="black"/>
-        </collision>
-        <inertial>
-            <mass value="0.01"/>
-            <inertia ixx="0.0" ixy="0.0" ixz="0.0" iyy="0.0" iyz="0.0" izz="0.0"/>
-        </inertial>
-    </link>
-    <!-- Back Bumper Link -->
-    <link name="BackBumper">
-        <visual>
-            <geometry>
-                <mesh filename="file://$(find junior_description)/meshes/robitBackBumper.stl"/>
-            </geometry>
-            <material name="black"/>
-        </visual>
-        <collision>
-            <geometry>
-                <mesh filename="file://$(find junior_description)/meshes/robitBackBumper.stl"/>
-            </geometry>
-            <material name="black"/>
-        </collision>
-        <inertial>
-            <mass value="0.01"/>
-            <inertia ixx="0.0" ixy="0.0" ixz="0.0" iyy="0.0" iyz="0.0" izz="0.0"/>
-        </inertial>
-    </link>
     <!-- Front Lidar Link -->
     <link name="FrontLidar">
@@ -168,23 +130,4 @@
         </inertial>
     </link>
-    <!-- Risers Link -->
-    <link name="Risers">
-        <visual>
-            <geometry>
-                <mesh filename="file://$(find junior_description)/meshes/robitRiserVisual.stl"/>
-            </geometry>
-            <material name="black"/>
-        </visual>
-        <collision>
-            <geometry>
-                <mesh filename="file://$(find junior_description)/meshes/robitRiserCollision.stl"/>
-            </geometry>
-            <material name="black"/>
-        </collision>
-        <inertial>
-            <mass value="0.01"/>
-            <inertia ixx="0.0" ixy="0.0" ixz="0.0" iyy="0.0" iyz="0.0" izz="0.0"/>
-        </inertial>
-    </link>
     <!-- Back Lidar Link -->
     <link name="BackLidar">
@@ -217,9 +160,10 @@
         <visual>
             <geometry>
-                <mesh filename="file://$(find junior_description)/meshes/robitWheel.stl"/>
+                <mesh filename="file://$(find junior_description)/meshes/robitWheel.dae"/>
                 <!-- <cylinder length="0.105" radius="0.1575"/> -->
             </geometry>
             <material name="black"/>
             <!-- <origin xyz="0 0 0" rpy="1.57079632679 0 0"/>  Comment Out for Mesh -->
+            <origin rpy="-3.14159265359 0 0"/>
         </visual>
         <collision>
@@ -252,5 +196,5 @@
         <visual>
             <geometry>
-                <mesh filename="file://$(find junior_description)/meshes/robitWheel.stl"/>
+                <mesh filename="file://$(find junior_description)/meshes/robitWheel.dae"/>
                 <!-- <cylinder length="0.105" radius="0.1575"/> -->
             </geometry>
@@ -287,9 +231,10 @@
         <visual>
             <geometry>
-                <mesh filename="file://$(find junior_description)/meshes/robitWheel.stl"/>
+                <mesh filename="file://$(find junior_description)/meshes/robitWheel.dae"/>
                 <!-- <cylinder length="0.105" radius="0.1575"/> -->
             </geometry>
             <material name="black"/>
             <!-- <origin xyz="0 0 0" rpy="1.57079632679 0 0"/>  Comment Out for Mesh -->
+            <origin rpy="-3.14159265359 0 0"/>
         </visual>
         <collision>
@@ -322,5 +267,5 @@
         <visual>
             <geometry>
-                <mesh filename="file://$(find junior_description)/meshes/robitWheel.stl"/>
+                <mesh filename="file://$(find junior_description)/meshes/robitWheel.dae"/>
                 <!-- <cylinder length="0.105" radius="0.1575"/> -->
             </geometry>
@@ -380,5 +325,5 @@
         <parent link="Chassis"/>
         <child link="BackCameraCase"/>
-        <origin xyz="-0.285 0 0.339"/>
+        <origin xyz="-0.285 0 0.311"/>
     </joint>
     <joint name="BackCameraStandJoint" type="fixed">
@@ -397,9 +342,4 @@
         <limit lower="-1" upper="1" effort="5" velocity="2"/> FOR REVOLUTE -->
     </joint>
-    <joint name="RisersJoint" type="fixed">
-        <parent link="Chassis"/>
-        <child link="Risers"/>
-        <origin xyz="-0.057 0 0.2655"/>
-    </joint>
     <joint name="BackLidarJoint" type="fixed">
         <parent link="BackCameraCase"/>
@@ -435,14 +375,4 @@
         <origin xyz="-0.193 -0.2635 -0.07" rpy="0 0 0"/>
         <axis xyz="0 1 0"/>
-    </joint>
-    <joint name="FrontBumperLoc" type="fixed">
-        <parent link="Chassis"/>
-        <child link="FrontBumper"/>
-        <origin xyz="0.321 0 0.025" rpy="0 0 0"/>
-    </joint>
-    <joint name="BackBumperLoc" type="fixed">
-        <parent link="Chassis"/>
-        <child link="BackBumper"/>
-        <origin xyz="-0.321 0 -0.0795" rpy="0 0 0"/>
     </joint>
     <!-- END OF JOINTS -->

Commit message: Updated Both Lidar Positions - Front Scan is Colliding with Chassis Collision Model

File: urdf/junior.urdf.xacro (robot description, xacro)
@@ -315,5 +315,5 @@
         <parent link="Chassis"/>
         <child link="FrontLidar"/>
-        <origin xyz="0.321 0 -0.0197"/>
+        <origin xyz="0.321 0 -0.098"/>
     </joint>
     <joint name="FrontLidarVision" type="fixed">
@@ -415,5 +415,5 @@
         <sensor name="laser" type="ray">
             <pose> 0 0 0 0 0 0 </pose>
-            <visualize>false</visualize> <!-- TURN TO TRUE WHEN TESTING THE LIDAR -->
+            <visualize>true</visualize> <!-- TURN TO TRUE WHEN TESTING THE LIDAR -->
             <update_rate>10</update_rate>
             <ray>
@@ -575,5 +575,5 @@
             <!-- Max Teleop Speeds
                 Forward Speed: 1.8 m/s
-                Reverse Speed: 0 m/s
+                Reverse Speed: 0.2 m/s
                 Left Turn Speed: 7 m/s
                 Right Turn Speed: 7 m/s

Commit message: Dual Lidars Working with New Collision Model

File: urdf/junior.urdf.xacro (robot description, xacro)
@@ -25,5 +25,5 @@
         <collision>
             <geometry>
-                <mesh filename="file://$(find junior_description)/meshes/robitChassisCollision.dae"/>
+                <mesh filename="file://$(find junior_description)/meshes/robitChassisCollision.stl"/>
                <!-- <box size="0.642 0.39 0.412"/> -->
             </geometry>
@@ -415,5 +415,5 @@
         <sensor name="laser" type="ray">
             <pose> 0 0 0 0 0 0 </pose>
-            <visualize>true</visualize> <!-- TURN TO TRUE WHEN TESTING THE LIDAR -->
+            <visualize>false</visualize> <!-- TURN TO TRUE WHEN TESTING THE LIDAR -->
             <update_rate>10</update_rate>
             <ray>
@@ -426,5 +426,5 @@
                 </scan>
                 <range>
-                    <min>0.2</min>
+                    <min>0.1</min>
                     <max>3</max>
                 </range>
