Commit message: Implemented Two Motor System - Driving Fully Functional

File: urdf/junior.urdf.xacro (robot description, xacro)
@@ -161,8 +161,6 @@
             <geometry>
                 <mesh filename="file://$(find junior_description)/meshes/robitWheel.dae"/>
-                <!-- <cylinder length="0.105" radius="0.1575"/> -->
-            </geometry>
-            <material name="black"/>
-            <!-- <origin xyz="0 0 0" rpy="1.57079632679 0 0"/>  Comment Out for Mesh -->
+            </geometry>
+            <material name="black"/>
             <origin rpy="-3.14159265359 0 0"/>
         </visual>
@@ -174,15 +172,4 @@
             <!-- <origin xyz="0 0 0" rpy="1.57079632679 0 0"/> -->
             <material name="black"/>
-            <surface>
-                <friction>
-                    <ode>
-                        <mu>0.7</mu>
-                        <mu2>0.7</mu2>
-                        <kp>1000000</kp>
-                        <kd>1.0</kd>
-                        <fdir>1 0 0</fdir>
-                    </ode>
-                </friction>
-            </surface>
         </collision>
         <inertial>
@@ -197,8 +184,6 @@
             <geometry>
                 <mesh filename="file://$(find junior_description)/meshes/robitWheel.dae"/>
-                <!-- <cylinder length="0.105" radius="0.1575"/> -->
-            </geometry>
-            <material name="black"/>
-            <!-- <origin xyz="0 0 0" rpy="1.57079632679 0 0"/>  Comment Out for Mesh -->
+            </geometry>
+            <material name="black"/>
         </visual>
         <collision>
@@ -209,15 +194,4 @@
             <!-- <origin xyz="0 0 0" rpy="1.57079632679 0 0"/> -->
             <material name="black"/>
-            <surface>
-                <friction>
-                    <ode>
-                        <mu>0.7</mu>
-                        <mu2>0.7</mu2>
-                        <kp>1000000</kp>
-                        <kd>1.0</kd>
-                        <fdir>1 0 0</fdir>
-                    </ode>
-                </friction>
-            </surface>
         </collision>
         <inertial>
@@ -232,8 +206,6 @@
             <geometry>
                 <mesh filename="file://$(find junior_description)/meshes/robitWheel.dae"/>
-                <!-- <cylinder length="0.105" radius="0.1575"/> -->
-            </geometry>
-            <material name="black"/>
-            <!-- <origin xyz="0 0 0" rpy="1.57079632679 0 0"/>  Comment Out for Mesh -->
+            </geometry>
+            <material name="black"/>
             <origin rpy="-3.14159265359 0 0"/>
         </visual>
@@ -245,15 +217,4 @@
             <!-- <origin xyz="0 0 0" rpy="1.57079632679 0 0"/> -->
             <material name="black"/>
-            <surface>
-                <friction>
-                    <ode>
-                        <mu>0.7</mu>
-                        <mu2>0.7</mu2>
-                        <kp>1000000</kp>
-                        <kd>1.0</kd>
-                        <fdir>1 0 0</fdir>
-                    </ode>
-                </friction>
-            </surface>
         </collision>
         <inertial>
@@ -268,8 +229,6 @@
             <geometry>
                 <mesh filename="file://$(find junior_description)/meshes/robitWheel.dae"/>
-                <!-- <cylinder length="0.105" radius="0.1575"/> -->
-            </geometry>
-            <material name="black"/>
-            <!-- <origin xyz="0 0 0" rpy="1.57079632679 0 0"/>  Comment Out for Mesh -->
+            </geometry>
+            <material name="black"/>
         </visual>
         <collision>
@@ -280,15 +239,4 @@
             <!-- <origin xyz="0 0 0" rpy="1.57079632679 0 0"/> -->
             <material name="black"/>
-            <surface>
-                <friction>
-                    <ode>
-                        <mu>0.7</mu>
-                        <mu2>0.7</mu2>
-                        <kp>1000000</kp>
-                        <kd>1.0</kd>
-                        <fdir>1 0 0</fdir>
-                    </ode>
-                </friction>
-            </surface>
         </collision>
         <inertial>
@@ -298,12 +246,4 @@
         </inertial>
     </link>
-    <!-- Graveyard of Wheel Inertias
-    Ted v1 : <inertia ixx="0.007" ixy="0.0" ixz="0.0" iyy="0.014" iyz="0.0" izz="0.007"/>
-    Cylinder Math : <inertia ixx="0.014" ixy="0.0" ixz="0.0" iyy="0.014" iyz="0.0" izz="0.024"/>
-    Box Math : <inertia ixx="0.0183" ixy="0.0" ixz="0.0" iyy="0.033" iyz="0.0" izz="0.033"/>
-    Logi v1 : <inertia ixx="0.014" ixy="0.0" ixz="0.0" iyy="0.04" iyz="0.0" izz="0.024"/>
-    CURRENT: Precision Cylinder : <inertia ixx="0.014240625" ixy="0.0" ixz="0.0" iyy="0.014240625" iyz="0.0" izz="0.02480625"/>
-    Gazebo Cylinder : <inertia ixx="0.15" ixy="0.0" ixz="0.0" iyy="0.15" iyz="0.0" izz="0.13"/>
-    -->
     <!-- START OF JOINTS -->
     <joint name="ChassisJoint" type="fixed">
@@ -380,24 +320,4 @@
     <!-- Chassis -->
     <gazebo reference="Chassis">
-    </gazebo>
-    <!-- Front Bumper -->
-    <gazebo reference="FrontBumper">
-        <visual>
-            <material>
-                <diffuse>0.2 0.2 0.2 1</diffuse>
-                <ambient>0.1 0.1 0.1 1</ambient>
-                <emissive>0 0 0 0</emissive>
-            </material>
-        </visual>
-    </gazebo>
-    <!-- Back Bumper -->
-    <gazebo reference="BackBumper">
-        <visual>
-            <material>
-                <diffuse>0.2 0.2 0.2 1</diffuse>
-                <ambient>0.1 0.1 0.1 1</ambient>
-                <emissive>0 0 0 0</emissive>
-            </material>
-        </visual>
     </gazebo>
     <!-- Front Lidar Case -->
@@ -456,5 +376,5 @@
         </visual>
     </gazebo>
-    <!-- Back Lidar Stand -->
+    <!-- Back Camera Stand -->
     <gazebo reference="BackCameraStand">
         <visual>
@@ -466,5 +386,5 @@
         </visual>
     </gazebo>
-    <!-- Back Lidar Head -->
+    <!-- Back Camera Head -->
     <gazebo reference="BackCameraHead">
         <visual>
@@ -472,14 +392,4 @@
                 <diffuse>0.77 0.78 0.78 1</diffuse>
                 <ambient>0.385 0.39 0.39 1</ambient>
-                <emissive>0 0 0 0</emissive>
-            </material>
-        </visual>
-    </gazebo>
-    <!-- Risers -->
-    <gazebo reference="Risers">
-        <visual>
-            <material>
-                <diffuse>0.2 0.2 0.2 1</diffuse>
-                <ambient>0.1 0.1 0.1 1</ambient>
                 <emissive>0 0 0 0</emissive>
             </material>
@@ -526,46 +436,78 @@
     <!-- WHEELS -->
     <gazebo reference="WheelLeftFront">
-        <visual>
-            <material>
-                <diffuse>0.2 0.2 0.2 1</diffuse>
-                <ambient>0.1 0.1 0.1 1</ambient>
-                <emissive>0 0 0 0</emissive>
-            </material>
-        </visual>
+        <collision>
+            <surface>
+                <friction>
+                    <ode>
+                        <mu>1.0</mu>
+                        <mu2>1.0</mu2>
+                        <kp>10000000</kp>
+                        <kd>1</kd>
+                    </ode>
+                </friction>
+            </surface>
+        </collision>
     </gazebo>
     <gazebo reference="WheelRightFront">
-        <visual>
-            <material>
-                <diffuse>0.2 0.2 0.2 1</diffuse>
-                <ambient>0.1 0.1 0.1 1</ambient>
-                <emissive>0 0 0 0</emissive>
-            </material>
-        </visual>
+        <collision>
+            <surface>
+                <friction>
+                    <ode>
+                        <mu>1.0</mu>
+                        <mu2>1.0</mu2>
+                        <kp>10000000</kp>
+                        <kd>1</kd>
+                    </ode>
+                </friction>
+            </surface>
+        </collision>
     </gazebo>
     <gazebo reference="WheelLeftBack">
-        <visual>
-            <material>
-                <diffuse>0.2 0.2 0.2 1</diffuse>
-                <ambient>0.1 0.1 0.1 1</ambient>
-                <emissive>0 0 0 0</emissive>
-            </material>
-        </visual>
+        <collision>
+            <surface>
+                <friction>
+                    <ode>
+                        <mu>1.0</mu>
+                        <mu2>1.0</mu2>
+                        <kp>10000000</kp>
+                        <kd>1</kd>
+                    </ode>
+                </friction>
+            </surface>
+        </collision>
     </gazebo>
     <gazebo reference="WheelRightBack">
-        <visual>
-            <material>
-                <diffuse>0.2 0.2 0.2 1</diffuse>
-                <ambient>0.1 0.1 0.1 1</ambient>
-                <emissive>0 0 0 0</emissive>
-            </material>
-        </visual>
+        <collision>
+            <surface>
+                <friction>
+                    <ode>
+                        <mu>1.0</mu>
+                        <mu2>1.0</mu2>
+                        <kp>10000000</kp>
+                        <kd>1</kd>
+                    </ode>
+                </friction>
+            </surface>
+        </collision>
     </gazebo>
     <!-- END OF WHEELS -->
     <gazebo>
-        <plugin name="diff_drive_controller" filename="libgazebo_ros_diff_drive.so">
-            <num_wheel_pairs>2</num_wheel_pairs>
+        <plugin name="diff_drive" filename="libgazebo_ros_diff_drive.so">
             <left_joint>AxleLeftFront</left_joint>
+            <right_joint>AxleRightFront</right_joint>
+            <wheel_separation>0.435</wheel_separation>
+            <wheel_diameter>0.315</wheel_diameter>
+            <max_wheel_torque>30.0</max_wheel_torque>
+            <max_wheel_acceleration>0.7</max_wheel_acceleration>
+            <odometry_frame>odom</odometry_frame>
+            <robot_base_frame>base_link</robot_base_frame>
+            <publish_odom>true</publish_odom>
+            <publish_odom_tf>true</publish_odom_tf>
+            <publish_wheel_tf>true</publish_wheel_tf>
+        </plugin>
+    </gazebo>
+    <gazebo>
+        <plugin name="diff_drive2" filename="libgazebo_ros_diff_drive.so">
             <left_joint>AxleLeftBack</left_joint>
-            <right_joint>AxleRightFront</right_joint>
             <right_joint>AxleRightBack</right_joint>
             <wheel_separation>0.435</wheel_separation>
@@ -573,10 +515,4 @@
             <max_wheel_torque>30.0</max_wheel_torque>
             <max_wheel_acceleration>0.7</max_wheel_acceleration>
-            <!-- Max Teleop Speeds
-                Forward Speed: 1.8 m/s
-                Reverse Speed: 0.06 m/s
-                Left Turn Speed: 1 m/s
-                Right Turn Speed: 1 m/s
-            -->
             <odometry_frame>odom</odometry_frame>
             <robot_base_frame>base_link</robot_base_frame>
@@ -584,7 +520,13 @@
             <publish_odom_tf>true</publish_odom_tf>
             <publish_wheel_tf>true</publish_wheel_tf>
-            <update_rate>100.0</update_rate>
         </plugin>
     </gazebo>
+    <!-- Max Teleop Speeds
+                Forward Speed: 1.8 m/s
+                Reverse Speed: 0.06 m/s
+                Left Turn Speed: 1 m/s
+                Right Turn Speed: 1 m/s
+                THESE STATS ARE WITH OLD ONE MOTOR SYSTEM
+    -->
     <!-- END OF GAZEBO -->
 </robot>

Commit message: Lidar Visual and Ray Changes

File: urdf/junior.urdf.xacro (robot description, xacro)
@@ -39,5 +39,5 @@
         <visual>
             <geometry>
-                <mesh filename="file://$(find junior_description)/meshes/robitFrontLidarCase.stl"/>
+                <mesh filename="file://$(find junior_description)/meshes/robitFrontLidarVisual.dae"/>
             </geometry>
             <material name="skyblue"/>
@@ -56,18 +56,6 @@
     <!-- Front Lidar Glass Link -->
     <link name="FrontLidarGlass">
-        <visual>
-            <geometry>
-                <mesh filename="file://$(find junior_description)/meshes/robitFrontLidarGlass.stl"/>
-            </geometry>
-            <material name="black"/>
-        </visual>
-        <collision>
-            <geometry>
-                <mesh filename="file://$(find junior_description)/meshes/robitFrontLidarGlass.stl"/>
-            </geometry>
-            <material name="black"/>
-        </collision>
-        <inertial>
-            <mass value="0.01"/>
+        <inertial>
+            <mass value="0.001"/>
             <inertia ixx="0.0" ixy="0.0" ixz="0.0" iyy="0.0" iyz="0.0" izz="0.0"/>
         </inertial>
@@ -167,8 +155,8 @@
         <collision>
             <geometry>
-                <mesh filename="file://$(find junior_description)/meshes/robitWheelCollision.dae"/>
-                <!-- <cylinder length="0.105" radius="0.1575"/> -->
-            </geometry>
-            <!-- <origin xyz="0 0 0" rpy="1.57079632679 0 0"/> -->
+                <!-- <mesh filename="file://$(find junior_description)/meshes/robitWheelCollision.dae"/> -->
+                <cylinder length="0.105" radius="0.1575"/>
+            </geometry>
+            <origin xyz="0 0 0" rpy="1.57079632679 0 0"/>
             <material name="black"/>
         </collision>
@@ -189,8 +177,8 @@
         <collision>
             <geometry>
-                <mesh filename="file://$(find junior_description)/meshes/robitWheelCollision.dae"/>
-                <!-- <cylinder length="0.105" radius="0.1575"/> -->
-            </geometry>
-            <!-- <origin xyz="0 0 0" rpy="1.57079632679 0 0"/> -->
+                <!-- <mesh filename="file://$(find junior_description)/meshes/robitWheelCollision.dae"/> -->
+                <cylinder length="0.105" radius="0.1575"/>
+            </geometry>
+            <origin xyz="0 0 0" rpy="1.57079632679 0 0"/>
             <material name="black"/>
         </collision>
@@ -212,8 +200,8 @@
         <collision>
             <geometry>
-                <mesh filename="file://$(find junior_description)/meshes/robitWheelCollision.dae"/>
-                <!-- <cylinder length="0.105" radius="0.1575"/> -->
-            </geometry>
-            <!-- <origin xyz="0 0 0" rpy="1.57079632679 0 0"/> -->
+                <!-- <mesh filename="file://$(find junior_description)/meshes/robitWheelCollision.dae"/> -->
+                <cylinder length="0.105" radius="0.1575"/>
+            </geometry>
+            <origin xyz="0 0 0" rpy="1.57079632679 0 0"/>
             <material name="black"/>
         </collision>
@@ -234,8 +222,8 @@
         <collision>
             <geometry>
-                <mesh filename="file://$(find junior_description)/meshes/robitWheelCollision.dae"/>
-                <!-- <cylinder length="0.105" radius="0.1575"/> -->
-            </geometry>
-            <!-- <origin xyz="0 0 0" rpy="1.57079632679 0 0"/> -->
+                <!-- <mesh filename="file://$(find junior_description)/meshes/robitWheelCollision.dae"/> -->
+                <cylinder length="0.105" radius="0.1575"/>
+            </geometry>
+            <origin xyz="0 0 0" rpy="1.57079632679 0 0"/>
             <material name="black"/>
         </collision>
@@ -255,10 +243,10 @@
         <parent link="Chassis"/>
         <child link="FrontLidar"/>
-        <origin xyz="0.321 0 -0.098"/>
+        <origin xyz="0.321 0 -0.085"/>
     </joint>
     <joint name="FrontLidarVision" type="fixed">
         <parent link="FrontLidar"/>
         <child link="FrontLidarGlass"/>
-        <origin xyz="0.075 0 0"/>
+        <origin xyz="0.08 0 -0.03"/>
     </joint>
     <joint name="BackCameraHolster" type="fixed">
@@ -290,5 +278,5 @@
         <parent link="BackLidar"/>
         <child link="BackLidarScanner"/>
-        <origin xyz="0 0 0.03" rpy="0 0 0"/>
+        <origin xyz="0 0 0.055" rpy="0 0 0"/>
     </joint>
     <joint name="AxleLeftFront" type="continuous">
@@ -323,11 +311,4 @@
     <!-- Front Lidar Case -->
     <gazebo reference="FrontLidar">
-        <visual>
-            <material>
-                <diffuse>0.1 0.5 1 1</diffuse>
-                <ambient>0.0666 0.333 0.4 1</ambient>
-                <emissive>0 0 0 0</emissive>
-            </material>
-        </visual>
     </gazebo>
     <!-- Front Lidar -->
@@ -358,11 +339,4 @@
             </plugin>
         </sensor>
-        <visual>
-            <material>
-                <diffuse>0.2 0.2 0.2 1</diffuse>
-                <ambient>0.1 0.1 0.1 1</ambient>
-                <emissive>0 0 0 0</emissive>
-            </material>
-        </visual>
     </gazebo>
     <!-- Back Camera Case -->
