Commit message: Updated Naming Conventions to be Consistent with Repository

File: urdf/junior.urdf.xacro (robot description, xacro)
@@ -20,10 +20,10 @@
         <visual>
             <geometry>
-                <mesh filename="file://$(find junior_description)/meshes/robitChassisVisual.dae"/>
-            </geometry>
-        </visual>
-        <collision>
-            <geometry>
-                <mesh filename="file://$(find junior_description)/meshes/robitChassisCollision.stl"/>
+                <mesh filename="file://$(find atrvjr_description)/meshes/robitChassisVisual.dae"/>
+            </geometry>
+        </visual>
+        <collision>
+            <geometry>
+                <mesh filename="file://$(find atrvjr_description)/meshes/robitChassisCollision.stl"/>
                <!-- <box size="0.642 0.39 0.412"/> -->
             </geometry>
@@ -39,5 +39,5 @@
         <visual>
             <geometry>
-                <mesh filename="file://$(find junior_description)/meshes/robitFrontLidarVisual.dae"/>
+                <mesh filename="file://$(find atrvjr_description)/meshes/robitFrontLidarVisual.dae"/>
             </geometry>
             <material name="skyblue"/>
@@ -45,5 +45,5 @@
         <collision>
             <geometry>
-                <mesh filename="file://$(find junior_description)/meshes/robitFrontLidarCase.stl"/>
+                <mesh filename="file://$(find atrvjr_description)/meshes/robitFrontLidarCase.stl"/>
             </geometry>
             <material name="skyblue"/>
@@ -65,11 +65,11 @@
         <visual>
             <geometry>
-                <mesh filename="file://$(find junior_description)/meshes/robitBackCameraCase.stl"/>
-            </geometry>
-            <material name="black"/>
-        </visual>
-        <collision>
-            <geometry>
-                <mesh filename="file://$(find junior_description)/meshes/robitBackCameraCase.stl"/>
+                <mesh filename="file://$(find atrvjr_description)/meshes/robitBackCameraCase.stl"/>
+            </geometry>
+            <material name="black"/>
+        </visual>
+        <collision>
+            <geometry>
+                <mesh filename="file://$(find atrvjr_description)/meshes/robitBackCameraCase.stl"/>
             </geometry>
             <material name="black"/>
@@ -84,5 +84,5 @@
         <visual>
             <geometry>
-                <mesh filename="file://$(find junior_description)/meshes/robitBackCameraStand.stl"/>
+                <mesh filename="file://$(find atrvjr_description)/meshes/robitBackCameraStand.stl"/>
             </geometry>
             <material name="silver"/>
@@ -90,5 +90,5 @@
         <collision>
             <geometry>
-                <mesh filename="file://$(find junior_description)/meshes/robitBackCameraStand.stl"/>
+                <mesh filename="file://$(find atrvjr_description)/meshes/robitBackCameraStand.stl"/>
             </geometry>
             <material name="silver"/>
@@ -103,5 +103,5 @@
         <visual>
             <geometry>
-                <mesh filename="file://$(find junior_description)/meshes/robitBackCameraHead.stl"/>
+                <mesh filename="file://$(find atrvjr_description)/meshes/robitBackCameraHead.stl"/>
             </geometry>
             <material name="silver"/>
@@ -109,5 +109,5 @@
         <collision>
             <geometry>
-                <mesh filename="file://$(find junior_description)/meshes/robitBackCameraHead.stl"/>
+                <mesh filename="file://$(find atrvjr_description)/meshes/robitBackCameraHead.stl"/>
             </geometry>
             <material name="silver"/>
@@ -122,11 +122,11 @@
         <visual>
             <geometry>
-                <mesh filename="file://$(find junior_description)/meshes/hokuyo_urg_04lx.dae"/>
-            </geometry>
-            <material name="black"/>
-        </visual>
-        <collision>
-            <geometry>
-                <mesh filename="file://$(find junior_description)/meshes/hokuyo_urg_04lx.dae"/>
+                <mesh filename="file://$(find atrvjr_description)/meshes/hokuyo_urg_04lx.dae"/>
+            </geometry>
+            <material name="black"/>
+        </visual>
+        <collision>
+            <geometry>
+                <mesh filename="file://$(find atrvjr_description)/meshes/hokuyo_urg_04lx.dae"/>
             </geometry>
             <material name="black"/>
@@ -148,5 +148,5 @@
         <visual>
             <geometry>
-                <mesh filename="file://$(find junior_description)/meshes/robitWheel.dae"/>
+                <mesh filename="file://$(find atrvjr_description)/meshes/robitWheel.dae"/>
             </geometry>
             <material name="black"/>
@@ -155,5 +155,5 @@
         <collision>
             <geometry>
-                <!-- <mesh filename="file://$(find junior_description)/meshes/robitWheelCollision.dae"/> -->
+                <!-- <mesh filename="file://$(find atrvjr_description)/meshes/robitWheelCollision.dae"/> -->
                 <cylinder length="0.105" radius="0.1575"/>
             </geometry>
@@ -171,11 +171,11 @@
         <visual>
             <geometry>
-                <mesh filename="file://$(find junior_description)/meshes/robitWheel.dae"/>
-            </geometry>
-            <material name="black"/>
-        </visual>
-        <collision>
-            <geometry>
-                <!-- <mesh filename="file://$(find junior_description)/meshes/robitWheelCollision.dae"/> -->
+                <mesh filename="file://$(find atrvjr_description)/meshes/robitWheel.dae"/>
+            </geometry>
+            <material name="black"/>
+        </visual>
+        <collision>
+            <geometry>
+                <!-- <mesh filename="file://$(find atrvjr_description)/meshes/robitWheelCollision.dae"/> -->
                 <cylinder length="0.105" radius="0.1575"/>
             </geometry>
@@ -193,5 +193,5 @@
         <visual>
             <geometry>
-                <mesh filename="file://$(find junior_description)/meshes/robitWheel.dae"/>
+                <mesh filename="file://$(find atrvjr_description)/meshes/robitWheel.dae"/>
             </geometry>
             <material name="black"/>
@@ -200,5 +200,5 @@
         <collision>
             <geometry>
-                <!-- <mesh filename="file://$(find junior_description)/meshes/robitWheelCollision.dae"/> -->
+                <!-- <mesh filename="file://$(find atrvjr_description)/meshes/robitWheelCollision.dae"/> -->
                 <cylinder length="0.105" radius="0.1575"/>
             </geometry>
@@ -216,11 +216,11 @@
         <visual>
             <geometry>
-                <mesh filename="file://$(find junior_description)/meshes/robitWheel.dae"/>
-            </geometry>
-            <material name="black"/>
-        </visual>
-        <collision>
-            <geometry>
-                <!-- <mesh filename="file://$(find junior_description)/meshes/robitWheelCollision.dae"/> -->
+                <mesh filename="file://$(find atrvjr_description)/meshes/robitWheel.dae"/>
+            </geometry>
+            <material name="black"/>
+        </visual>
+        <collision>
+            <geometry>
+                <!-- <mesh filename="file://$(find atrvjr_description)/meshes/robitWheelCollision.dae"/> -->
                 <cylinder length="0.105" radius="0.1575"/>
             </geometry>

Commit message: Back Camera Fully Functional

File: urdf/junior.urdf.xacro (robot description, xacro)
@@ -118,4 +118,11 @@
         </inertial>
     </link>
+    <!-- Back Camera Visual Link -->
+    <link name="BackCameraVisual">
+        <inertial>
+            <mass value="0.001"/>
+            <inertia ixx="0.0" ixy="0.0" ixz="0.0" iyy="0.0" iyz="0.0" izz="0.0"/>
+        </inertial>
+    </link>
     <!-- Back Lidar Link -->
     <link name="BackLidar">
@@ -269,4 +276,9 @@
         <!-- <dynamics damping="0" friction="0.75"/>
         <limit lower="-1" upper="1" effort="5" velocity="2"/> FOR REVOLUTE -->
+    </joint>
+    <joint name="BackCameraVisualJoint" type="fixed">
+        <parent link="BackCameraHead"/>
+        <child link="BackCameraVisual"/>
+        <origin xyz="0.07 0 0" rpy="0 0 0"/>
     </joint>
     <joint name="BackLidarJoint" type="fixed">
@@ -369,4 +381,39 @@
             </material>
         </visual>
+    </gazebo>
+    <!-- Back Camera Visual -->
+    <gazebo reference="BackCameraVisual">
+        <sensor name="bcamera" type="camera">
+            <pose>0 0 0 0 0 0</pose>
+            <camera>
+                <horizontal_fov>2.0</horizontal_fov>
+                <image>
+                    <format>R8G8B8</format>
+                    <width>640</width>
+                    <height>360</height>
+                </image>
+                <clip>
+                    <near>0.05</near>
+                    <far>15000</far>
+                </clip>
+            </camera>
+            <always_on>1</always_on>
+            <update_rate>30</update_rate>
+            <visualize>false</visualize>
+            <plugin name="camera_controller" filename="libgazebo_ros_camera.so">
+                <alwaysOn>true</alwaysOn>
+                <updateRate>0.0</updateRate>
+                <cameraName>bcamera</cameraName>
+                <imageTopicName>bimage_raw</imageTopicName>
+                <cameraInfoTopicName>bcamera_info</cameraInfoTopicName>
+                <frameName>camera_link</frameName>
+                <hackBaseline>0.07</hackBaseline>
+                <distortionK1>0.0</distortionK1>
+                <distortionK2>0.0</distortionK2>
+                <distortionK3>0.0</distortionK3>
+                <distortionT1>0.0</distortionT1>
+                <distortionT2>0.0</distortionT2>
+            </plugin>
+        </sensor>
     </gazebo>
     <!-- Back Lidar -->

Commit message: Added Optional Orbital Camera

File: urdf/junior.urdf.xacro (robot description, xacro)
@@ -35,4 +35,11 @@
         </inertial>
     </link>
+    <!-- Test Orbital Cam
+    <link name="OrbitalCamera">
+        <inertial>
+            <mass value="0.001"/>
+            <inertia ixx="0.0" ixy="0.0" ixz="0.0" iyy="0.0" iyz="0.0" izz="0.0"/>
+        </inertial>
+    </link> -->
     <!-- Front Lidar Link -->
     <link name="FrontLidar">
@@ -247,4 +254,9 @@
         <origin xyz="0 0 0.23"/>
     </joint>
+    <!-- <joint name="OrbitalCamera" type="fixed">
+        <parent link="Chassis"/>
+        <child link="OrbitalCamera"/>
+        <origin xyz="0 0 3" rpy="0 1.57 0"/>
+    </joint> -->
     <joint name="FrontLidarHolster" type="fixed">
         <parent link="Chassis"/>
@@ -321,4 +333,38 @@
     <gazebo reference="Chassis">
     </gazebo>
+    <!-- <gazebo reference="OrbitalCamera">
+        <sensor name="ocamera" type="camera">
+            <pose>0 0 0 0 0 0</pose>
+            <camera>
+                <horizontal_fov>1.0</horizontal_fov>
+                <image>
+                    <format>R8G8B8</format>
+                    <width>700</width>
+                    <height>700</height>
+                </image>
+                <clip>
+                    <near>0.01</near>
+                    <far>15000</far>
+                </clip>
+            </camera>
+            <always_on>1</always_on>
+            <update_rate>30</update_rate>
+            <visualize>false</visualize>
+            <plugin name="ocamera_controller" filename="libgazebo_ros_camera.so">
+                <alwaysOn>true</alwaysOn>
+                <updateRate>0.0</updateRate>
+                <cameraName>ocamera</cameraName>
+                <imageTopicName>oimage_raw</imageTopicName>
+                <cameraInfoTopicName>ocamera_info</cameraInfoTopicName>
+                <frameName>camera_link</frameName>
+                <hackBaseline>0.07</hackBaseline>
+                <distortionK1>0.0</distortionK1>
+                <distortionK2>0.0</distortionK2>
+                <distortionK3>0.0</distortionK3>
+                <distortionT1>0.0</distortionT1>
+                <distortionT2>0.0</distortionT2>
+            </plugin>
+        </sensor>
+    </gazebo> -->
     <!-- Front Lidar Case -->
     <gazebo reference="FrontLidar">
